File: S3-Kicad/GPIO.sch (KiCad schematic (older format))
At the start: 100 parts, among them J1 Conn_01x04, J2 Conn_02x16_Counter_Clockwise, U1 74HC574, U2 74HC541, U3 74HC574, U4 74HC541, U5 74HC574, U6 74HC541, U7 74HC574, U8 74HC541, U9 74HC574

Commit message: Circuit Board Drafted (it could probably be improved)
Parts:
- removed J1: Conn_01x04, Connector_PinHeader_2.54mm:PinHeader_1x04_P2.54mm_Vertical, symbol Connector_Generic:Conn_01x04
- removed J2: Conn_02x16_Counter_Clockwise, Connector_PinHeader_2.54mm:PinHeader_2x15_P2.54mm_Vertical, symbol Connector_Generic:Conn_02x16_Counter_Clockwise
- added J7: Conn_02x16_Odd_Even, Connector_PinHeader_2.54mm:PinHeader_2x16_P2.54mm_Vertical, symbol Connector_Generic:Conn_02x16_Odd_Even
- renumbered R33 to R19, R34 to R20, R19 to R21, R20 to R22, R21 to R23, R22 to R24, R35 to R25, R36 to R26, R23 to R27, R24 to R28, R25 to R29, R26 to R30, R27 to R31, R28 to R32, R29 to R33, R30 to R34, R31 to R35, R32 to R36, R115 to R37, R116 to R38, R117 to R39, R118 to R40, R119 to R41, R120 to R42, R121 to R43, R122 to R44, R37 to R45, R38 to R46, R123 to R47, R124 to R48, R39 to R49, R40 to R50, R125 to R51, R126 to R52, R127 to R53, R128 to R54, R41 to R55, R42 to R56, R43 to R57, R44 to R58, R45 to R59, R46 to R60, R47 to R61, R48 to R62, R49 to R63, U8 to U10, U9 to U11, U1 to U3, U2 to U4, U3 to U5, U4 to U6, U5 to U7, U6 to U8, U7 to U9
Connections:
- net P0: now also J7.1 (Pin_1)
- net P1: now also J7.3 (Pin_3)
- net P10: now also J7.21 (Pin_21)
- net P11: now also J7.23 (Pin_23)
- net P12: now also J7.25 (Pin_25)
- net P13: now also J7.27 (Pin_27)
- net P14: now also J7.29 (Pin_29)
- net P15: now also J7.31 (Pin_31)
- net P16: now also J7.32 (Pin_32)
- net P17: now also J7.30 (Pin_30)
- net P18: now also J7.28 (Pin_28)
- net P19: now also J7.26 (Pin_26)
- net P2: now also J7.5 (Pin_5)
- net P20: now also J7.24 (Pin_24)
- net P21: now also J7.22 (Pin_22)
- net P22: now also J7.20 (Pin_20)
- net P23: now also J7.18 (Pin_18)
- net P24: now also J7.16 (Pin_16)
- net P25: now also J7.14 (Pin_14)
- net P26: now also J7.12 (Pin_12)
- net P27: now also J7.10 (Pin_10)
- net P28: now also J7.8 (Pin_8)
- net P29: now also J7.6 (Pin_6)
- net P3: now also J7.7 (Pin_7)
- net P30: now also J7.4 (Pin_4)
- net P31: now also J7.2 (Pin_2)
- net P4: now also J7.9 (Pin_9)
- net P5: now also J7.11 (Pin_11)
- net P6: now also J7.13 (Pin_13)
- net P7: now also J7.15 (Pin_15)
- net P8: now also J7.17 (Pin_17)
- net P9: now also J7.19 (Pin_19)
- net FLASHPAGE2: now reaches D37.2 (A), U11.15 (Q4)
- net FLASHPAGE1: now reaches D38.2 (A), U11.14 (Q5)
- net FLASHPAGE0: now reaches D39.2 (A), U11.13 (Q6)
- net RAM_PAGE: now reaches D40.2 (A), U11.12 (Q7)
