File: S3-Kicad/Memory.sch (KiCad schematic (older format))
At the start: 7 parts, among them U28 CY62136EV30LL-45ZSXI

Commit message: Circuit Board Drafted (it could probably be improved)
Parts:
- removed R88: 50K, Resistor_SMD:R_0805_2012Metric, symbol Device:R
- renumbered R83 to R113, R84 to R114, R85 to R115, R86 to R116, R87 to R117, U28 to U30
Connections:
- net RAM_PAGE: now reaches U30.24 (A11)
Changed lines of the file:
@@
 $Descr A4 11693 8268
 encoding utf-8
-Sheet 6 8
+Sheet 6 9
 Title ""
 Date ""
@@
 P 5350 2850
 AR Path="/667002CD" Ref="U?"  Part="1"
-AR Path="/635D7970/667002CD" Ref="U28"  Part="1"
-F 0 "U28" H 5950 3115 50  0000 C CNN
+AR Path="/635D7970/667002CD" Ref="U30"  Part="1"
+F 0 "U30" H 5950 3115 50  0000 C CNN
 F 1 "CY62136EV30LL-45ZSXI" H 5950 3024 50  0000 C CNN
 F 2 "Package_SO:TSOP-II-44_10.16x18.41mm_P0.8mm" H 5750 3550 50  0001 L CNN
@@
 $Comp
 L Device:R R?
-U 1 1 667002B1
-P 6700 4850
-AR Path="/667002B1" Ref="R?"  Part="1"
-AR Path="/635D7970/667002B1" Ref="R88"  Part="1"
-F 0 "R88" V 6600 4750 50  0000 C CNN
-F 1 "50K" V 6600 4900 50  0000 C CNN
-F 2 "Resistor_SMD:R_0805_2012Metric" V 6630 4850 50  0001 C CNN
-F 3 "~" H 6700 4850 50  0001 C CNN
-	1    6700 4850
-	0    -1   -1   0
-$EndComp
-$Comp
-L Device:R R?
 U 1 1 667002AB
 P 6800 3150
 AR Path="/667002AB" Ref="R?"  Part="1"
-AR Path="/635D7970/667002AB" Ref="R83"  Part="1"
-F 0 "R83" V 6800 2700 50  0000 C CNN
+AR Path="/635D7970/667002AB" Ref="R113"  Part="1"
+F 0 "R113" V 6800 2700 50  0000 C CNN
 F 1 "50K" V 6800 2850 50  0000 C CNN
 F 2 "Resistor_SMD:R_0805_2012Metric" V 6730 3150 50  0001 C CNN
@@
 P 6800 3250
 AR Path="/667002A5" Ref="R?"  Part="1"
-AR Path="/635D7970/667002A5" Ref="R84"  Part="1"
-F 0 "R84" V 6800 2800 50  0000 C CNN
+AR Path="/635D7970/667002A5" Ref="R114"  Part="1"
+F 0 "R114" V 6800 2800 50  0000 C CNN
 F 1 "50K" V 6800 2950 50  0000 C CNN
 F 2 "Resistor_SMD:R_0805_2012Metric" V 6730 3250 50  0001 C CNN
@@
 P 6800 3350
 AR Path="/6670029F" Ref="R?"  Part="1"
-AR Path="/635D7970/6670029F" Ref="R86"  Part="1"
-F 0 "R86" V 6800 2900 50  0000 C CNN
+AR Path="/635D7970/6670029F" Ref="R116"  Part="1"
+F 0 "R116" V 6800 2900 50  0000 C CNN
 F 1 "50K" V 6800 3050 50  0000 C CNN
 F 2 "Resistor_SMD:R_0805_2012Metric" V 6730 3350 50  0001 C CNN
@@
 P 5100 3350
 AR Path="/66700299" Ref="R?"  Part="1"
-AR Path="/635D7970/66700299" Ref="R85"  Part="1"
-F 0 "R85" V 5100 2900 50  0000 C CNN
+AR Path="/635D7970/66700299" Ref="R115"  Part="1"
+F 0 "R115" V 5100 2900 50  0000 C CNN
 F 1 "50K" V 5100 3050 50  0000 C CNN
 F 2 "Resistor_SMD:R_0805_2012Metric" V 5030 3350 50  0001 C CNN
@@
 P 5100 4450
 AR Path="/66700293" Ref="R?"  Part="1"
-AR Path="/635D7970/66700293" Ref="R87"  Part="1"
-F 0 "R87" V 5100 4000 50  0000 C CNN
+AR Path="/635D7970/66700293" Ref="R117"  Part="1"
+F 0 "R117" V 5100 4000 50  0000 C CNN
 F 1 "50K" V 5100 4150 50  0000 C CNN
 F 2 "Resistor_SMD:R_0805_2012Metric" V 5030 4450 50  0001 C CNN
@@
 Wire Wire Line
 	6950 3250 6950 3350
-Wire Wire Line
-	6950 4850 6850 4850
 Connection ~ 6950 3350
 Wire Wire Line
@@
 P 7000 3150
 AR Path="/6670027E" Ref="#PWR?"  Part="1"
-AR Path="/635D7970/6670027E" Ref="#PWR0169"  Part="1"
-F 0 "#PWR0169" H 7000 3000 50  0001 C CNN
+AR Path="/635D7970/6670027E" Ref="#PWR079"  Part="1"
+F 0 "#PWR079" H 7000 3000 50  0001 C CNN
 F 1 "+3.3V" H 7015 3323 50  0000 C CNN
 F 2 "" H 7000 3150 50  0001 C CNN
@@
 P 6950 4850
 AR Path="/66700277" Ref="#PWR?"  Part="1"
-AR Path="/635D7970/66700277" Ref="#PWR0168"  Part="1"
-F 0 "#PWR0168" H 6950 4600 50  0001 C CNN
+AR Path="/635D7970/66700277" Ref="#PWR082"  Part="1"
+F 0 "#PWR082" H 6950 4600 50  0001 C CNN
 F 1 "GND" H 6955 4677 50  0000 C CNN
 F 2 "" H 6950 4850 50  0001 C CNN
@@
 	1    0    0    -1
 $EndComp
-Connection ~ 6950 4850
 Wire Wire Line
 	5350 3950 5050 3950
@@
 P 5050 4050
 AR Path="/66700269" Ref="#PWR?"  Part="1"
-AR Path="/635D7970/66700269" Ref="#PWR0167"  Part="1"
-F 0 "#PWR0167" H 5050 3800 50  0001 C CNN
+AR Path="/635D7970/66700269" Ref="#PWR081"  Part="1"
+F 0 "#PWR081" H 5050 3800 50  0001 C CNN
 F 1 "GND" H 5055 3877 50  0000 C CNN
 F 2 "" H 5050 4050 50  0001 C CNN
@@
 P 4900 3250
 AR Path="/66700260" Ref="#PWR?"  Part="1"
-AR Path="/635D7970/66700260" Ref="#PWR0166"  Part="1"
-F 0 "#PWR0166" H 4900 3100 50  0001 C CNN
+AR Path="/635D7970/66700260" Ref="#PWR080"  Part="1"
+F 0 "#PWR080" H 4900 3100 50  0001 C CNN
 F 1 "+3.3V" H 4915 3423 50  0000 C CNN
 F 2 "" H 4900 3250 50  0001 C CNN
@@
 Wire Notes Line
 	4400 2500 7450 2500
+Text GLabel 6700 5300 0    50   Input ~ 0
+RAM_PAGE
+Wire Wire Line
+	6550 4850 6700 4850
+Wire Wire Line
+	6700 4850 6700 5300
 Wire Bus Line
 	2950 2750 2950 4350
