File: S3-Kicad/MicroCodeDecoder.sch (KiCad schematic (older format))
At the start: 32 parts, among them U10 SST39VF800A-70-4C-EKE, U11 74HC541, U12 74HC541, U13 74HC541, U14 74HC541, U15 74HC00

Commit message: Circuit Board Drafted (it could probably be improved)
Parts:
- renumbered R50 to R64, R51 to R65, R52 to R66, R53 to R67, R54 to R68, R55 to R69, R56 to R70, R57 to R71, R58 to R72, R59 to R73, R60 to R74, R61 to R75, R62 to R76, R63 to R77, R64 to R78, R65 to R79, R66 to R80, R67 to R81, R68 to R82, R69 to R83, R70 to R84, R71 to R85, R72 to R86, R73 to R87, R74 to R88, R75 to R89, U10 to U12, U11 to U13, U12 to U14, U13 to U15, U14 to U16, U15 to U17
Connections:
- net JumpS2 is gone; now on net ~CounterOutEnable: U12.35 (DQ3)
- net ~CounterOutEnable: no longer U17.3
- net ~RamAddrEnable: no longer U17.2
- net ~StackOut: no longer U17.1
- net JumpS1 renamed FlashOut
- no-connect marks 19 -> 22
Other:
- moved on the sheet: U17D
