File: S3-Kicad/ProgramCounter.sch (KiCad schematic (older format))
At the start: 43 parts, among them J9 Conn_01x16, U16 74hc193, U17 74hc193, U18 74hc193, U19 74hc193, U20 74HC541, U21 74HC541

Commit message: Circuit Board Drafted (it could probably be improved)
Parts:
- renumbered J9 to J8, R76 to R100, R139 to R101, R77 to R102, R78 to R103, R140 to R104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
