File: S3-Kicad/Registers.sch (KiCad schematic (older format))
At the start: 0 parts

Commit message: Schematic Done
Parts:
- added R100, R101, R102, R103, R104, R105, R106, R107, R108, R109, R110, R111, R112, R89, R90, R91, R92, R93, R94, R95, R96, R97, R98, R99: 50K, Resistor_SMD:R_0805_2012Metric, symbol Device:R
- added U29, U30, U31, U32, U33, U34, U35, U36, U37, U38, U39, U40, U41, U42, U43, U44: 74HC574, Package_SO:TSSOP-20_4.4x6.5mm_P0.65mm, symbol S3_Schematic-rescue:74LS573-74xx-MAX7000CPU-Gen2-rescue
- added U45, U46, U47, U48, U49, U50, U51, U52, U53, U54, U55, U56, U57, U58, U59, U60: 74HC541, Package_SO:TSSOP-20_4.4x6.5mm_P0.65mm, symbol 74xx:74LS541
Connections:
- new net: R98.1, U38.1 (OE)
- new net: R97.1, U37.1 (OE)
- new net: R90.1, U30.1 (OE)
- new net: R104.1, U44.1 (OE)
- new net: R103.1, U43.1 (OE)
- new net: R96.1, U36.1 (OE)
- new net: R95.1, U35.1 (OE)
- new net +3V3: R100.2, R101.2, R102.2, R105.1, R106.1, R107.1, R108.1, R109.1, R110.1, R111.1, R112.1, R91.2, R92.2, R93.2, R94.2, R99.2, U29.20 (VCC), U30.20 (VCC), U31.20 (VCC), U32.20 (VCC), U33.20 (VCC), U34.20 (VCC), U35.20 (VCC), U36.20 (VCC), U37.20 (VCC), U38.20 (VCC), U39.20 (VCC), U40.20 (VCC), U41.20 (VCC), U42.20 (VCC), U43.20 (VCC), U44.20 (VCC), U45.20 (VCC), U46.20 (VCC), U47.20 (VCC), U48.20 (VCC), U49.20 (VCC), U50.20 (VCC), U51.20 (VCC), U52.20 (VCC), U53.20 (VCC), U54.20 (VCC), U55.20 (VCC), U56.20 (VCC), U57.20 (VCC), U58.20 (VCC), U59.20 (VCC), U60.20 (VCC)
- new net Acc0: U30.19 (Q0), U45.2 (A0), U47.2 (A0), U49.2 (A0)
- new net Acc1: U30.18 (Q1), U45.3 (A1), U47.3 (A1), U49.3 (A1)
- new net Acc10: U38.17 (Q2), U46.4 (A2), U48.4 (A2), U50.4 (A2)
- new net Acc11: U38.16 (Q3), U46.5 (A3), U48.5 (A3), U50.5 (A3)
- new net Acc12: U38.15 (Q4), U46.6 (A4), U48.6 (A4), U50.6 (A4)
- new net Acc13: U38.14 (Q5), U46.7 (A5), U48.7 (A5), U50.7 (A5)
- new net Acc14: U38.13 (Q6), U46.8 (A6), U48.8 (A6), U50.8 (A6)
- new net Acc15: U38.12 (Q7), U46.9 (A7), U48.9 (A7), U50.9 (A7)
- new net Acc2: U30.17 (Q2), U45.4 (A2), U47.4 (A2), U49.4 (A2)
- new net Acc3: U30.16 (Q3), U45.5 (A3), U47.5 (A3), U49.5 (A3)
- new net Acc4: U30.15 (Q4), U45.6 (A4), U47.6 (A4), U49.6 (A4)
- new net Acc5: U30.14 (Q5), U45.7 (A5), U47.7 (A5), U49.7 (A5)
- new net Acc6: U30.13 (Q6), U45.8 (A6), U47.8 (A6), U49.8 (A6)
- new net Acc7: U30.12 (Q7), U45.9 (A7), U47.9 (A7), U49.9 (A7)
- new net Acc8: U38.19 (Q0), U46.2 (A0), U48.2 (A0), U50.2 (A0)
- new net Acc9: U38.18 (Q1), U46.3 (A1), U48.3 (A1), U50.3 (A1)
- new net B0: U29.2 (D0), U30.2 (D0), U31.2 (D0), U32.2 (D0), U33.2 (D0), U34.2 (D0), U35.2 (D0), U36.2 (D0), U45.18 (Y0)
- new net B1: U29.3 (D1), U30.3 (D1), U31.3 (D1), U32.3 (D1), U33.3 (D1), U34.3 (D1), U35.3 (D1), U36.3 (D1), U45.17 (Y1)
- new net B10: U37.4 (D2), U38.4 (D2), U39.4 (D2), U40.4 (D2), U41.4 (D2), U42.4 (D2), U43.4 (D2), U44.4 (D2), U46.16 (Y2)
- new net B11: U37.5 (D3), U38.5 (D3), U39.5 (D3), U40.5 (D3), U41.5 (D3), U42.5 (D3), U43.5 (D3), U44.5 (D3), U46.15 (Y3)
- new net B12: U37.6 (D4), U38.6 (D4), U39.6 (D4), U40.6 (D4), U41.6 (D4), U42.6 (D4), U43.6 (D4), U44.6 (D4), U46.14 (Y4)
- new net B13: U37.7 (D5), U38.7 (D5), U39.7 (D5), U40.7 (D5), U41.7 (D5), U42.7 (D5), U43.7 (D5), U44.7 (D5), U46.13 (Y5)
- new net B14: U37.8 (D6), U38.8 (D6), U39.8 (D6), U40.8 (D6), U41.8 (D6), U42.8 (D6), U43.8 (D6), U44.8 (D6), U46.12 (Y6)
- new net B15: U37.9 (D7), U38.9 (D7), U39.9 (D7), U40.9 (D7), U41.9 (D7), U42.9 (D7), U43.9 (D7), U44.9 (D7), U46.11 (Y7)
- new net B2: U29.4 (D2), U30.4 (D2), U31.4 (D2), U32.4 (D2), U33.4 (D2), U34.4 (D2), U35.4 (D2), U36.4 (D2), U45.16 (Y2)
- new net B3: U29.5 (D3), U30.5 (D3), U31.5 (D3), U32.5 (D3), U33.5 (D3), U34.5 (D3), U35.5 (D3), U36.5 (D3), U45.15 (Y3)
- new net B4: U29.6 (D4), U30.6 (D4), U31.6 (D4), U32.6 (D4), U33.6 (D4), U34.6 (D4), U35.6 (D4), U36.6 (D4), U45.14 (Y4)
- new net B5: U29.7 (D5), U30.7 (D5), U31.7 (D5), U32.7 (D5), U33.7 (D5), U34.7 (D5), U35.7 (D5), U36.7 (D5), U45.13 (Y5)
- new net B6: U29.8 (D6), U30.8 (D6), U31.8 (D6), U32.8 (D6), U33.8 (D6), U34.8 (D6), U35.8 (D6), U36.8 (D6), U45.12 (Y6)
- new net B7: U29.9 (D7), U30.9 (D7), U31.9 (D7), U32.9 (D7), U33.9 (D7), U34.9 (D7), U35.9 (D7), U36.9 (D7), U45.11 (Y7)
- new net B8: U37.2 (D0), U38.2 (D0), U39.2 (D0), U40.2 (D0), U41.2 (D0), U42.2 (D0), U43.2 (D0), U44.2 (D0), U46.18 (Y0)
- new net B9: U37.3 (D1), U38.3 (D1), U39.3 (D1), U40.3 (D1), U41.3 (D1), U42.3 (D1), U43.3 (D1), U44.3 (D1), U46.17 (Y1)
- new net EvenR0: U32.19 (Q0), U34.19 (Q0), U49.18 (Y0), U53.18 (Y0), U57.18 (Y0)
- new net EvenR1: U32.18 (Q1), U34.18 (Q1), U49.17 (Y1), U53.17 (Y1), U57.17 (Y1)
- new net EvenR10: U40.17 (Q2), U42.17 (Q2), U50.16 (Y2), U54.16 (Y2), U58.16 (Y2)
- new net EvenR11: U40.16 (Q3), U42.16 (Q3), U50.15 (Y3), U54.15 (Y3), U58.15 (Y3)
- new net EvenR12: U40.15 (Q4), U42.15 (Q4), U50.14 (Y4), U54.14 (Y4), U58.14 (Y4)
- new net EvenR13: U40.14 (Q5), U42.14 (Q5), U50.13 (Y5), U54.13 (Y5), U58.13 (Y5)
- new net EvenR14: U40.13 (Q6), U42.13 (Q6), U50.12 (Y6), U54.12 (Y6), U58.12 (Y6)
- new net EvenR15: U40.12 (Q7), U42.12 (Q7), U50.11 (Y7), U54.11 (Y7), U58.11 (Y7)
- new net EvenR2: U32.17 (Q2), U34.17 (Q2), U49.16 (Y2), U53.16 (Y2), U57.16 (Y2)
- new net EvenR3: U32.16 (Q3), U34.16 (Q3), U49.15 (Y3), U53.15 (Y3), U57.15 (Y3)
- new net EvenR4: U32.15 (Q4), U34.15 (Q4), U49.14 (Y4), U53.14 (Y4), U57.14 (Y4)
- new net EvenR5: U32.14 (Q5), U34.14 (Q5), U49.13 (Y5), U53.13 (Y5), U57.13 (Y5)
- new net EvenR6: U32.13 (Q6), U34.13 (Q6), U49.12 (Y6), U53.12 (Y6), U57.12 (Y6)
- new net EvenR7: U32.12 (Q7), U34.12 (Q7), U49.11 (Y7), U53.11 (Y7), U57.11 (Y7)
- new net EvenR8: U40.19 (Q0), U42.19 (Q0), U50.18 (Y0), U54.18 (Y0), U58.18 (Y0)
- new net EvenR9: U40.18 (Q1), U42.18 (Q1), U50.17 (Y1), U54.17 (Y1), U58.17 (Y1)
- new net GND: R103.2, R104.2, R89.2, R90.2, R95.2, R96.2, R97.2, R98.2, U29.10 (GND), U30.10 (GND), U31.10 (GND), U32.10 (GND), U33.10 (GND), U34.10 (GND), U35.10 (GND), U36.10 (GND), U37.10 (GND), U38.10 (GND), U39.10 (GND), U40.10 (GND), U41.10 (GND), U42.10 (GND), U43.10 (GND), U44.10 (GND), U45.10 (GND), U46.10 (GND), U47.10 (GND), U48.10 (GND), U49.10 (GND), U50.10 (GND), U51.10 (GND), U52.10 (GND), U53.10 (GND), U54.10 (GND), U55.10 (GND), U56.10 (GND), U57.10 (GND), U58.10 (GND), U59.10 (GND), U60.10 (GND)
- new net Ins0: U29.19 (Q0)
- new net Ins1: U29.18 (Q1)
- new net Ins10: U37.17 (Q2)
- new net Ins11: U37.16 (Q3)
- new net Ins12: U37.15 (Q4)
- new net Ins13: U37.14 (Q5)
- new net Ins14: U37.13 (Q6)
- new net Ins15: U37.12 (Q7)
- new net Ins2: U29.17 (Q2)
- new net Ins3: U29.16 (Q3)
- new net Ins4: U29.15 (Q4)
- new net Ins5: U29.14 (Q5)
- new net Ins6: U29.13 (Q6)
- new net Ins7: U29.12 (Q7)
- new net Ins8: U37.19 (Q0)
- new net Ins9: U37.18 (Q1)
- new net InsRegControl: U29.11 (Load), U37.11 (Load)
- new net JB0: U35.19 (Q0), U57.2 (A0), U59.2 (A0)
- new net JB1: U35.18 (Q1), U57.3 (A1), U59.3 (A1)
- new net JB10: U43.17 (Q2), U58.4 (A2), U60.4 (A2)
- new net JB11: U43.16 (Q3), U58.5 (A3), U60.5 (A3)
- new net JB12: U43.15 (Q4), U58.6 (A4), U60.6 (A4)
- new net JB13: U43.14 (Q5), U58.7 (A5), U60.7 (A5)
- new net JB14: U43.13 (Q6), U58.8 (A6), U60.8 (A6)
- new net JB15: U43.12 (Q7), U58.9 (A7), U60.9 (A7)
- new net JB2: U35.17 (Q2), U57.4 (A2), U59.4 (A2)
- new net JB3: U35.16 (Q3), U57.5 (A3), U59.5 (A3)
- new net JB4: U35.15 (Q4), U57.6 (A4), U59.6 (A4)
- new net JB5: U35.14 (Q5), U57.7 (A5), U59.7 (A5)
- new net JB6: U35.13 (Q6), U57.8 (A6), U59.8 (A6)
- new net JB7: U35.12 (Q7), U57.9 (A7), U59.9 (A7)
- new net JB8: U43.19 (Q0), U58.2 (A0), U60.2 (A0)
- new net JB9: U43.18 (Q1), U58.3 (A1), U60.3 (A1)
- new net MA0: U51.18 (Y0)
- new net MA1: U51.17 (Y1)
- new net MA10: U52.16 (Y2)
- new net MA11: U52.15 (Y3)
- new net MA12: U52.14 (Y4)
- new net MA13: U52.13 (Y5)
- new net MA14: U52.12 (Y6)
- new net MA15: U52.11 (Y7)
- new net MA2: U51.16 (Y2)
- new net MA3: U51.15 (Y3)
- new net MA4: U51.14 (Y4)
- new net MA5: U51.13 (Y5)
- new net MA6: U51.12 (Y6)
- new net MA7: U51.11 (Y7)
- new net MA8: U52.18 (Y0)
- new net MA9: U52.17 (Y1)
- new net MainRegReadControl: U30.11 (Load), U38.11 (Load)
- new net OddR0: U31.19 (Q0), U33.19 (Q0), U47.18 (Y0), U55.18 (Y0), U59.18 (Y0)
- new net OddR1: U31.18 (Q1), U33.18 (Q1), U47.17 (Y1), U55.17 (Y1), U59.17 (Y1)
- new net OddR10: U39.17 (Q2), U41.17 (Q2), U48.16 (Y2), U56.16 (Y2), U60.16 (Y2)
- new net OddR11: U39.16 (Q3), U41.16 (Q3), U48.15 (Y3), U56.15 (Y3), U60.15 (Y3)
- new net OddR12: U39.15 (Q4), U41.15 (Q4), U48.14 (Y4), U56.14 (Y4), U60.14 (Y4)
- new net OddR13: U39.14 (Q5), U41.14 (Q5), U48.13 (Y5), U56.13 (Y5), U60.13 (Y5)
- new net OddR14: U39.13 (Q6), U41.13 (Q6), U48.12 (Y6), U56.12 (Y6), U60.12 (Y6)
- new net OddR15: U39.12 (Q7), U41.12 (Q7), U48.11 (Y7), U56.11 (Y7), U60.11 (Y7)
- new net OddR2: U31.17 (Q2), U33.17 (Q2), U47.16 (Y2), U55.16 (Y2), U59.16 (Y2)
- new net OddR3: U31.16 (Q3), U33.16 (Q3), U47.15 (Y3), U55.15 (Y3), U59.15 (Y3)
- new net OddR4: U31.15 (Q4), U33.15 (Q4), U47.14 (Y4), U55.14 (Y4), U59.14 (Y4)
- new net OddR5: U31.14 (Q5), U33.14 (Q5), U47.13 (Y5), U55.13 (Y5), U59.13 (Y5)
- new net OddR6: U31.13 (Q6), U33.13 (Q6), U47.12 (Y6), U55.12 (Y6), U59.12 (Y6)
- new net OddR7: U31.12 (Q7), U33.12 (Q7), U47.11 (Y7), U55.11 (Y7), U59.11 (Y7)
- new net OddR8: U39.19 (Q0), U41.19 (Q0), U48.18 (Y0), U56.18 (Y0), U60.18 (Y0)
- new net OddR9: U39.18 (Q1), U41.18 (Q1), U48.17 (Y1), U56.17 (Y1), U60.17 (Y1)
- new net ProgramInsDisable: R89.1, U29.1 (OE)
- new net R1Control: U31.11 (Load), U39.11 (Load)
- new net R2Control: U32.11 (Load), U40.11 (Load)
- new net R3Control: U33.11 (Load), U41.11 (Load)
- new net R4Control: U34.11 (Load), U42.11 (Load)
- new net RA0: U36.19 (Q0), U51.2 (A0), U53.2 (A0), U55.2 (A0)
- new net RA1: U36.18 (Q1), U51.3 (A1), U53.3 (A1), U55.3 (A1)
- new net RA10: U44.17 (Q2), U52.4 (A2), U54.4 (A2), U56.4 (A2)
- new net RA11: U44.16 (Q3), U52.5 (A3), U54.5 (A3), U56.5 (A3)
- new net RA12: U44.15 (Q4), U52.6 (A4), U54.6 (A4), U56.6 (A4)
- new net RA13: U44.14 (Q5), U52.7 (A5), U54.7 (A5), U56.7 (A5)
- new net RA14: U44.13 (Q6), U52.8 (A6), U54.8 (A6), U56.8 (A6)
- new net RA15: U44.12 (Q7), U52.9 (A7), U54.9 (A7), U56.9 (A7)
- new net RA2: U36.17 (Q2), U51.4 (A2), U53.4 (A2), U55.4 (A2)
- new net RA3: U36.16 (Q3), U51.5 (A3), U53.5 (A3), U55.5 (A3)
- new net RA4: U36.15 (Q4), U51.6 (A4), U53.6 (A4), U55.6 (A4)
- new net RA5: U36.14 (Q5), U51.7 (A5), U53.7 (A5), U55.7 (A5)
- new net RA6: U36.13 (Q6), U51.8 (A6), U53.8 (A6), U55.8 (A6)
- new net RA7: U36.12 (Q7), U51.9 (A7), U53.9 (A7), U55.9 (A7)
- new net RA8: U44.19 (Q0), U52.2 (A0), U54.2 (A0), U56.2 (A0)
- new net RA9: U44.18 (Q1), U52.3 (A1), U54.3 (A1), U56.3 (A1)
- new net RJBControl: U35.11 (Load), U43.11 (Load)
- new net RMAControl: U36.11 (Load), U44.11 (Load)
- new net ~MainRegLeftOutput: R106.2, U47.1 (G1), U47.19 (G2), U48.1 (G1), U48.19 (G2)
- new net ~MainRegOutputControl: R105.2, U45.1 (G1), U45.19 (G2), U46.1 (G1), U46.19 (G2)
- new net ~MainRegRightOutput: R107.2, U49.1 (G1), U49.19 (G2), U50.1 (G1), U50.19 (G2)
- new net ~R1Out: R91.1, R99.1, U31.1 (OE), U39.1 (OE)
- new net ~R2Out: R100.1, R92.1, U32.1 (OE), U40.1 (OE)
- new net ~R3Out: R101.1, R93.1, U33.1 (OE), U41.1 (OE)
- new net ~R4Out: R102.1, R94.1, U34.1 (OE), U42.1 (OE)
- new net ~RJBLeftOutput: R112.2, U59.1 (G1), U59.19 (G2), U60.1 (G1), U60.19 (G2)
- new net ~RJBRightOutput: R111.2, U57.1 (G1), U57.19 (G2), U58.1 (G1), U58.19 (G2)
- new net ~RMALeftOutput: R110.2, U55.1 (G1), U55.19 (G2), U56.1 (G1), U56.19 (G2)
- new net ~RMARightOutput: R109.2, U53.1 (G1), U53.19 (G2), U54.1 (G1), U54.19 (G2)
- new net ~RamAddrEnable: R108.2, U51.1 (G1), U51.19 (G2), U52.1 (G1), U52.19 (G2)
Other:
- note added: "General Purpose Registers/Control"

Commit message: Circuit Board Drafted (it could probably be improved)
Parts:
- renumbered R89 to R118, R90 to R119, R91 to R120, R92 to R121, R93 to R122, R94 to R123, R95 to R124, R96 to R125, R97 to R126, R98 to R127, R99 to R128, R100 to R129, R101 to R130, R102 to R131, R103 to R132, R104 to R133, R105 to R134, R106 to R135, R107 to R136, R108 to R137, R109 to R138, R110 to R139, R111 to R140, R112 to R141, U29 to U31, U30 to U32, U31 to U33, U32 to U34, U33 to U35, U34 to U36, U35 to U37, U36 to U38, U37 to U39, U38 to U40, U39 to U41, U40 to U42, U41 to U43, U42 to U44, U43 to U45, U44 to U46, U45 to U47, U46 to U48, U47 to U49, U48 to U50, U49 to U51, U50 to U52, U51 to U53, U52 to U54, U53 to U55, U54 to U56, U55 to U57, U56 to U58, U57 to U59, U58 to U60, U59 to U61, U60 to U62
