File: S3-Kicad/S3_Schematic.kicad_pcb (KiCad board)
At the start: 2 copper layers, 160 x 100 mm, 345 parts, among them J1 Conn_01x04, J10 Conn_01x16, J11 Conn_01x16, J2 Conn_02x16_Counter_Clockwise, J3 Conn_02x04_Counter_Clockwise, J4 Conn_01x02, J5 Conn_01x02, J6 Conn_01x04, J7 Conn_01x04, J8 Conn_01x03, J9 Conn_01x16, U1 74HC574, U10 SST39VF800A-70-4C-EKE, U11 74HC541, U12 74HC541, U13 74HC541, U14 74HC541, U15 74HC00, U16 74hc193, U17 74hc193, U18 74hc193, U19 74hc193, U2 74HC541, U20 74HC541, U21 74HC541, U22 74hc193, U23 74hc193, U24 74hc193, U25 74hc193, U26 74HC541, U27 74HC541, U28 CY62136EV30LL-45ZSXI, U29 74HC574, U3 74HC574, U30 74HC574, U31 74HC574, U32 74HC574, U33 74HC574, U34 74HC574, U35 74HC574, U36 74HC574, U37 74HC574, U38 74HC574, U39 74HC574, U4 74HC541, U40 74HC574, U41 74HC574, U42 74HC574, U43 74HC574, U44 74HC574, U45 74HC541, U46 74HC541, U47 74HC541, U48 74HC541, U49 74HC541, U5 74HC574, U50 74HC541, U51 74HC541, U52 74HC541, U53 74HC541, U54 74HC541, U55 74HC541, U56 74HC541, U57 74HC541, U58 74HC541, U59 74HC541, U6 74HC541, U60 74HC541, U61 XC9572XL-10TQG100C, U62 SN74LVC1GX04DCKR, U63 74HC541, U7 74HC574, U8 74HC541, U9 74HC574, Y1 Crystal

Commit message: Circuit Board Drafted (it could probably be improved)
Parts:
- removed C36, C40, C47, C52, C53, C58, C64, C69: 100, Capacitor_SMD:C_0805_2012Metric
- removed the J2 at (115.5, -114.7)
- removed the J3 at (193.5, -108.0)
- removed the J6 at (206.4, -114.7)
- removed the R112 at (169.9, -48.3)
- removed the R114 at (61.2, -115.5)
- removed the R115 at (171.2, -100.7)
- removed the R116 at (153.7, -83.6)
- removed the R117 at (149.2, -78.4)
- removed the R118 at (175.7, -106.7)
- removed the R119 at (149.2, -81.3)
- removed the R121 at (162.5, -94.6)
- removed the R125 at (171.2, -103.6)
- removed the R126 at (162.5, -97.5)
- removed the R127 at (175.7, -109.6)
- removed the R129 at (47.0, -47.4)
- removed the R131 at (38.2, -46.4)
- removed the R133 at (51.6, -49.4)
- removed the R134 at (60.5, -52.4)
- removed the R136 at (51.4, -43.5)
- removed the R137 at (38.2, -41.5)
- removed the R64 at (51.2, 0.30)
- removed the R65 at (59.9, -7.50)
- removed the R66 at (51.2, -2.65)
- removed the R67 at (73.2, -22.1)
- removed the R76 at (38.2, -32.6)
- removed the R77 at (38.2, -60.1)
- removed the R88 at (127.3, -23.3)
- removed the U10 at (225.0, -26.0)
- removed the U13 at (66.6, -19.6)
- removed the U16 at (66.6, -66.3)
- removed the U31 at (132.7, -49.5)
- removed the U38 at (141.4, -49.5)
- removed the U39 at (124.0, -49.5)
- removed the U47 at (150.2, -33.4)
- removed the U48 at (158.9, -57.5)
- removed the U53 at (158.9, -65.6)
- removed the U54 at (141.4, -33.4)
- added C71: 100n, Capacitor_SMD:C_0805_2012Metric, B.Cu at (132.6, 63.5)
- added C72: 100n, Capacitor_SMD:C_0805_2012Metric, B.Cu at (173.0, 82.4)
- added C73: 100n, Capacitor_SMD:C_0805_2012Metric, B.Cu at (145.1, 63.5)
- added C74: 100n, Capacitor_SMD:C_0805_2012Metric, B.Cu at (79.8, 109.9)
- added C75: 100n, Capacitor_SMD:C_0805_2012Metric, B.Cu at (214.0, 89.6)
- added C76: 100n, Capacitor_SMD:C_0805_2012Metric, B.Cu at (199.7, 108.6)
- added C77: 100n, Capacitor_SMD:C_0805_2012Metric, B.Cu at (79.8, 116.9)
- added C78: 100n, Capacitor_SMD:C_0805_2012Metric, F.Cu at (181.8, 95.2)
- added J4: Conn_01x04, Connector_PinHeader_2.54mm:PinHeader_1x04_P2.54mm_Vertical, F.Cu at (207.2, 146.1)
- added J5: Conn_01x04, Connector_PinHeader_2.54mm:PinHeader_1x04_P2.54mm_Vertical, F.Cu at (224.9, 146.1)
- added R100: 50K, Resistor_SMD:R_0805_2012Metric, F.Cu at (113.8, 44.6)
- added R102: 50K, Resistor_SMD:R_0805_2012Metric, F.Cu at (113.8, 40.3)
- added R104: 330, Resistor_SMD:R_0805_2012Metric, B.Cu at (85.8, 35.0)
- added R105: 330, Resistor_SMD:R_0805_2012Metric, B.Cu at (82.7, 35.0)
- added R107: 330, Resistor_SMD:R_0805_2012Metric, B.Cu at (76.2, 35.0)
- added R108: 330, Resistor_SMD:R_0805_2012Metric, B.Cu at (73.0, 35.0)
- added R145: 50K, Resistor_SMD:R_0805_2012Metric, B.Cu at (138.1, 107.1)
- added R146: 50K, Resistor_SMD:R_0805_2012Metric, B.Cu at (145.1, 104.3)
- added R147: 50K, Resistor_SMD:R_0805_2012Metric, B.Cu at (138.2, 104.1)
- added R148: 50K, Resistor_SMD:R_0805_2012Metric, B.Cu at (141.9, 104.1)
- added R150: 50K, Resistor_SMD:R_0805_2012Metric, F.Cu at (129.2, 104.4)
- added R151: 50K, Resistor_SMD:R_0805_2012Metric, F.Cu at (173.1, 56.6)
- added R152: 50K, Resistor_SMD:R_0805_2012Metric, F.Cu at (170.1, 56.6)
- added R153: 50K, Resistor_SMD:R_0805_2012Metric, F.Cu at (167.2, 56.6)
- added R50: 50K, Resistor_SMD:R_0805_2012Metric, F.Cu at (215.9, 34.0)
- added R51: 330, Resistor_SMD:R_0805_2012Metric, B.Cu at (253.2, 97.8)
- added R52: 330, Resistor_SMD:R_0805_2012Metric, B.Cu at (248.2, 37.6)
- added R53: 330, Resistor_SMD:R_0805_2012Metric, B.Cu at (253.2, 102.4)
- added R61: 50K, Resistor_SMD:R_0805_2012Metric, B.Cu at (214.0, 87.0)
- added R62: 330, Resistor_SMD:R_0805_2012Metric, F.Cu at (230.0, 97.6)
- added R63: 330, Resistor_SMD:R_0805_2012Metric, F.Cu at (225.3, 97.6)
- added R68: 50K, Resistor_SMD:R_0805_2012Metric, B.Cu at (168.8, 100.1)
- added R69: 50K, Resistor_SMD:R_0805_2012Metric, F.Cu at (182.7, 62.6)
- added R70: 50K, Resistor_SMD:R_0805_2012Metric, B.Cu at (182.7, 63.9)
- added R71: 50K, Resistor_SMD:R_0805_2012Metric, F.Cu at (182.7, 65.5)
- added R72: 50K, Resistor_SMD:R_0805_2012Metric, B.Cu at (182.7, 67.2)
- added R73: 50K, Resistor_SMD:R_0805_2012Metric, F.Cu at (182.7, 68.9)
- added R74: 50K, Resistor_SMD:R_0805_2012Metric, B.Cu at (182.7, 70.6)
- added R90: 330, Resistor_SMD:R_0805_2012Metric, B.Cu at (120.9, 35.0)
- added R92: 330, Resistor_SMD:R_0805_2012Metric, B.Cu at (114.4, 35.0)
- added R96: 330, Resistor_SMD:R_0805_2012Metric, B.Cu at (101.4, 35.0)
- added R97: 330, Resistor_SMD:R_0805_2012Metric, B.Cu at (98.2, 35.0)
- added R98: 330, Resistor_SMD:R_0805_2012Metric, B.Cu at (95.5, 35.0)
- added U14: 74HC541, Package_SO:TSSOP-20_4.4x6.5mm_P0.65mm, F.Cu at (188.8, 76.3)
- added U27: 74hc193, Package_SO:TSSOP-16_4.4x5mm_P0.65mm, F.Cu at (79.8, 93.3)
- added U28: 74HC541, Package_SO:TSSOP-20_4.4x6.5mm_P0.65mm, F.Cu at (79.8, 67.0)
- added U37: 74HC574, Package_SO:TSSOP-20_4.4x6.5mm_P0.65mm, F.Cu at (105.1, 63.4)
- added U40: 74HC574, Package_SO:TSSOP-20_4.4x6.5mm_P0.65mm, F.Cu at (214.7, 102.3)
- added U43: 74HC574, Package_SO:TSSOP-20_4.4x6.5mm_P0.65mm, F.Cu at (123.7, 135.8)
- added U51: 74HC541, Package_SO:TSSOP-20_4.4x6.5mm_P0.65mm, F.Cu at (199.5, 111.3)
- added U52: 74HC541, Package_SO:TSSOP-20_4.4x6.5mm_P0.65mm, F.Cu at (199.3, 102.8)
- added U62: 74HC541, Package_SO:TSSOP-20_4.4x6.5mm_P0.65mm, F.Cu at (76.6, 135.8)
- added U63: XC9572XL-10TQG100C, Package_QFP:TQFP-100_14x14mm_P0.5mm, F.Cu at (127.5, 87.3)
- added U64: 74hc193, Package_SO:TSSOP-16_4.4x5mm_P0.65mm, F.Cu at (140.0, 104.3)
- added U65: SST39VF800A-70-4C-EKE, Package_SO:TSOP-I-48_18.4x12mm_P0.5mm, B.Cu at (175.7, 45.7)
- C10, C11, C12, C13, C14, C15, C16, C18, C19, C20, C21, C22, C23, C24, C25, C26, C27, C28, C29, C30, C31, C32, C33, C34, C35, C38, C39, C4, C41, C43, C44, C45, C48, C49, C5, C50, C51, C54, C56, C57, C59, C6, C60, C61, C62, C63, C65, C66, C67, C68, C7, C8, C9: value 100 -> 100n; moved to B.Cu
- C17, C3, C37, C42, C46, C55: value 100 -> 100n
- C70, R109, R111, R15, R16, R17, R18, R21, R22, R23, R24, R27, R28, R29, R30, R31, R32, R41, R42, R43, R44, R48: moved to B.Cu
- J1: value Conn_01x04 -> Conn_02x04_Counter_Clockwise; footprint Connector_PinHeader_2.54mm:PinHeader_1x04_P2.54mm_Vertical -> Connector_PinHeader_2.54mm:PinHeader_2x04_P2.54mm_Vertical
- J7: value Conn_01x04 -> Conn_02x16_Odd_Even; footprint Connector_PinHeader_2.54mm:PinHeader_1x04_P2.54mm_Vertical -> Connector_PinHeader_2.54mm:PinHeader_2x16_P2.54mm_Vertical
- R101, R106, R33, R34, R35, R36, R37, R38, R39, R40, R47, R54, R91, R93, R94, R95, R99: value 50K -> 330; moved to B.Cu
- R112: renamed from R82; value 50k -> 50K
- R113: renamed from R83; value 50k -> 50K
- R114: renamed from R84; value 50k -> 50K
- R115: renamed from R85; value 50k -> 50K; moved to B.Cu
- R116: renamed from R86; value 50k -> 50K
- R117: renamed from R87; value 50k -> 50K; moved to B.Cu
- R119: renamed from R90; moved to B.Cu
- R120, R122, R123, R124, R128, R130, R132, R135, R138, R139, R140, R141, R142, R143, R144: value 330 -> 50K; moved to B.Cu
- R121: renamed from R92; moved to B.Cu
- R125: renamed from R96; moved to B.Cu
- R127: renamed from R98; moved to B.Cu
- R129: renamed from R100; moved to B.Cu
- R131: renamed from R102; moved to B.Cu
- R133: renamed from R104; moved to B.Cu
- R134: renamed from R105; moved to B.Cu
- R136: renamed from R107; moved to B.Cu
- R14, R78, R79: value 50k -> 50K
- R19, R20, R25, R26, R45, R46, R49: value 330 -> 50K
- R55, R56, R57, R58, R59, R60: value 50K -> 330
- R64: renamed from R50; moved to B.Cu
- R65: renamed from R51; moved to B.Cu
- R66: renamed from R52; moved to B.Cu
- R67: renamed from R53; moved to B.Cu
- R75: renamed from R61; moved to B.Cu
- R76: renamed from R62; moved to B.Cu
- R77: renamed from R63; moved to B.Cu
- R80, R81: value 50k -> 50K; moved to B.Cu
- R82: renamed from R68; moved to B.Cu
- R83: renamed from R69; moved to B.Cu
- R84: renamed from R70; moved to B.Cu
- R85: renamed from R71; moved to B.Cu
- R86: renamed from R72; moved to B.Cu
- R87: renamed from R73; moved to B.Cu
- R88: renamed from R74; moved to B.Cu
- R89: renamed from R75; moved to B.Cu
- U12: value 74HC541 -> SST39VF800A-70-4C-EKE; footprint Package_SO:TSSOP-20_4.4x6.5mm_P0.65mm -> Package_SO:TSOP-I-48_18.4x12mm_P0.5mm
- U15: value 74HC00 -> 74HC541; footprint Package_SO:TSSOP-14_4.4x5mm_P0.65mm -> Package_SO:TSSOP-20_4.4x6.5mm_P0.65mm
- U17: value 74hc193 -> 74HC00; footprint Package_SO:TSSOP-16_4.4x5mm_P0.65mm -> Package_SO:TSSOP-14_4.4x5mm_P0.65mm; moved to B.Cu
- U20, U21, U26: value 74HC541 -> 74hc193; footprint Package_SO:TSSOP-20_4.4x6.5mm_P0.65mm -> Package_SO:TSSOP-16_4.4x5mm_P0.65mm
- U22, U23: value 74hc193 -> 74HC541; footprint Package_SO:TSSOP-16_4.4x5mm_P0.65mm -> Package_SO:TSSOP-20_4.4x6.5mm_P0.65mm
- U31: renamed from U29; moved to B.Cu
- U39: renamed from U37; moved to B.Cu
- U61: value XC9572XL-10TQG100C -> 74HC541; footprint Package_QFP:TQFP-100_14x14mm_P0.5mm -> Package_SO:TSSOP-20_4.4x6.5mm_P0.65mm
- moved C65 305.1 mm to (74.2, 135.8), turned to 90 degrees
- moved C54 295.3 mm to (87.6, 135.8), turned to 90 degrees
- moved C28 286.3 mm to (101.0, 135.8), turned to 90 degrees
- moved J1 284.9 mm to (250.9, 139.8), turned to 180 degrees
- moved C23 281.5 mm to (114.4, 135.8), turned to 90 degrees
- moved C39 281.2 mm to (107.7, 135.8), turned to 90 degrees
- moved C41 268.9 mm to (126.1, 135.8), turned to 90 degrees
- moved J3 261.2 mm to (239.3, 145.9), turned to 90 degrees
- moved C62 260.0 mm to (152.9, 135.8), turned to 90 degrees
- moved C48 258.1 mm to (79.8, 95.5)
- moved C63 257.9 mm to (172.8, 135.8), turned to 90 degrees
- moved R122 256.5 mm to (132.8, 135.8), turned to 270 degrees
- moved C15 252.4 mm to (179.5, 135.8), turned to 90 degrees
- moved J10 251.6 mm to (138.8, 116.0), turned to 90 degrees
- moved R8 248.7 mm to (230.3, 141.8), turned to 90 degrees
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- renumbered J11 to J10, J4 to J2, J5 to J3, J8 to J6, J9 to J8, J10 to J9, R89 to R118, R97 to R126, R108 to R137, R113 to R149, U62 to U1, U8 to U10, U9 to U11, U11 to U13, U14 to U16, U63 to U2, U27 to U29, U1 to U3, U28 to U30, U30 to U32, U32 to U34, U34 to U36, U36 to U38, U2 to U4, U40 to U42, U42 to U44, U43 to U45, U44 to U46, U45 to U47, U46 to U48, U3 to U5, U51 to U53, U52 to U54, U4 to U6, U5 to U7, U6 to U8, U7 to U9
Connections:
- D37 pad 2: Net-(D37-Pad2) -> FLASHPAGE2
- D38 pad 2: Net-(D38-Pad2) -> FLASHPAGE1
- D39 pad 2: Net-(D39-Pad2) -> FLASHPAGE0
- D40 pad 2: Net-(D40-Pad2) -> RAM_PAGE
- J1 pad 1: Net-(D37-Pad2) -> TMS_5V
- J1 pad 2: Net-(D38-Pad2) -> TDI_5V
- J1 pad 3: Net-(D39-Pad2) -> TDO_5V
- J1 pad 4: Net-(D40-Pad2) -> TCK_5V
- J7 pad 1: GND -> /GPIO/P0
- J7 pad 2: GND -> /GPIO/P31
- J7 pad 3: GND -> /GPIO/P1
- J7 pad 4: GND -> /GPIO/P30
- R101 pad 1: ~R3Out -> Net-(D51-Pad1)
- R101 pad 2: +3V3 -> GND
- R103 pad 1: Net-(R103-Pad1) -> GND
- R103 pad 2: GND -> CounterClear
- R106 pad 1: +3V3 -> Net-(D54-Pad1)
- R106 pad 2: ~MainRegLeftOutput -> GND
- R109 pad 1: +3V3 -> ~CounterOutEnable
- R109 pad 2: ~RMARightOutput -> +3V3
- R110 pad 2: ~RMALeftOutput -> ~StackLoad
- R111 pad 1: +3V3 -> GND
- R111 pad 2: ~RJBRightOutput -> StackClear
- R120 pad 1: Net-(D24-Pad1) -> ~R1Out
- R120 pad 2: GND -> +3V3
- R122 pad 1: Net-(D26-Pad1) -> ~R3Out
- R122 pad 2: GND -> +3V3
- R123 pad 1: Net-(D27-Pad1) -> ~R4Out
- R123 pad 2: GND -> +3V3
- R124 pad 1: Net-(D28-Pad1) -> Net-(R124-Pad1)
- R128 pad 1: Net-(D32-Pad1) -> ~R1Out
- R128 pad 2: GND -> +3V3
- R130 pad 1: Net-(D42-Pad1) -> ~R3Out
- R130 pad 2: GND -> +3V3
- R132 pad 1: Net-(D44-Pad1) -> Net-(R132-Pad1)
- R135 pad 1: Net-(D47-Pad1) -> +3V3
- R135 pad 2: GND -> ~MainRegLeftOutput
- R138 pad 1: Net-(D50-Pad1) -> +3V3
- R138 pad 2: GND -> ~RMARightOutput
- R139 pad 1: Net-(D51-Pad1) -> +3V3
- R139 pad 2: GND -> ~RMALeftOutput
- R140 pad 1: Net-(D52-Pad1) -> +3V3
- R140 pad 2: GND -> ~RJBRightOutput
- R141 pad 1: Net-(D53-Pad1) -> +3V3
- R141 pad 2: GND -> ~RJBLeftOutput
- R142 pad 1: Net-(D54-Pad1) -> +3V3
- R142 pad 2: GND -> Net-(R142-Pad2)
- R143 pad 1: Net-(D55-Pad1) -> +3V3
- R143 pad 2: GND -> Net-(R143-Pad2)
- R144 pad 1: Net-(D56-Pad1) -> +3V3
- R144 pad 2: GND -> Net-(R144-Pad2)
- R19 pad 1: Net-(D5-Pad1) -> +3V3
- R19 pad 2: GND -> ~PortAReadLow
- R20 pad 1: Net-(D6-Pad1) -> +3V3
- R20 pad 2: GND -> ~PortBReadLow
- R21 pad 1: Net-(D7-Pad1) -> Net-(D5-Pad1)
- R22 pad 1: Net-(D8-Pad1) -> Net-(D6-Pad1)
- R23 pad 1: Net-(D9-Pad1) -> Net-(D7-Pad1)
- R24 pad 1: Net-(D10-Pad1) -> Net-(D8-Pad1)
- R25 pad 1: Net-(D11-Pad1) -> +3V3
- R25 pad 2: GND -> ~ALDD
- R26 pad 1: Net-(D12-Pad1) -> +3V3
- R26 pad 2: GND -> ~BLDD
- R27 pad 1: Net-(D13-Pad1) -> Net-(D9-Pad1)
- R28 pad 1: Net-(D14-Pad1) -> Net-(D10-Pad1)
- R29 pad 1: Net-(D15-Pad1) -> Net-(D11-Pad1)
- R30 pad 1: Net-(D16-Pad1) -> Net-(D12-Pad1)
- R31 pad 1: Net-(D17-Pad1) -> Net-(D13-Pad1)
- R32 pad 1: Net-(D18-Pad1) -> Net-(D14-Pad1)
- R33 pad 1: +3V3 -> Net-(D15-Pad1)
- R33 pad 2: ~PortAReadLow -> GND
- R34 pad 1: +3V3 -> Net-(D16-Pad1)
- R34 pad 2: ~PortBReadLow -> GND
- R35 pad 1: +3V3 -> Net-(D17-Pad1)
- R35 pad 2: ~ALDD -> GND
- R36 pad 1: +3V3 -> Net-(D18-Pad1)
- R36 pad 2: ~BLDD -> GND
- R37 pad 1: +3V3 -> Net-(D19-Pad1)
- R37 pad 2: ~PortAReadHigh -> GND
- R38 pad 1: +3V3 -> Net-(D20-Pad1)
- R38 pad 2: ~PortBReadHigh -> GND
- R39 pad 1: +3V3 -> Net-(D21-Pad1)
- R39 pad 2: ~AHDD -> GND
- R40 pad 1: +3V3 -> Net-(D22-Pad1)
- R40 pad 2: ~BHDD -> GND
- R41 pad 1: Net-(D33-Pad1) -> Net-(D23-Pad1)
- R42 pad 1: Net-(D34-Pad1) -> Net-(D24-Pad1)
- R43 pad 1: Net-(D35-Pad1) -> Net-(D25-Pad1)
- R44 pad 1: Net-(D36-Pad1) -> Net-(D26-Pad1)
- R45 pad 1: Net-(D37-Pad1) -> +3V3
- R45 pad 2: GND -> ~PortAReadHigh
- R46 pad 1: Net-(D38-Pad1) -> +3V3
- R46 pad 2: GND -> ~PortBReadHigh
- R47 pad 1: GND -> Net-(D27-Pad1)
- R47 pad 2: Net-(R47-Pad2) -> GND
- R48 pad 1: Net-(D39-Pad1) -> Net-(D28-Pad1)
- R49 pad 1: Net-(D40-Pad1) -> +3V3
- R49 pad 2: GND -> ~AHDD
- R54 pad 1: GND -> Net-(D32-Pad1)
- R54 pad 2: PortAWriteLow -> GND
- R55 pad 1: GND -> Net-(D33-Pad1)
- R55 pad 2: RMAControl -> GND
- R56 pad 1: GND -> Net-(D34-Pad1)
- R56 pad 2: RJBControl -> GND
- R57 pad 1: GND -> Net-(D35-Pad1)
- R57 pad 2: R4Control -> GND
- R58 pad 1: GND -> Net-(D36-Pad1)
- R58 pad 2: R3Control -> GND
- R59 pad 1: GND -> Net-(D37-Pad1)
- R59 pad 2: R2Control -> GND
- R60 pad 1: GND -> Net-(D38-Pad1)
- R60 pad 2: R1Control -> GND
- R64 pad 2: Net-(R50-Pad2) -> Net-(R64-Pad2)
- R76 pad 2: Net-(R62-Pad2) -> Net-(R76-Pad2)
- R77 pad 2: Net-(R63-Pad2) -> Net-(R77-Pad2)
- R78 pad 1: GND -> +3V3
- R78 pad 2: CounterClear -> ~PortAReadLow
- R79 pad 1: ~CounterOutEnable -> +3V3
- R79 pad 2: +3V3 -> ~PortAReadHigh
- R80 pad 2: ~StackLoad -> ~PortBReadLow
- R81 pad 1: GND -> +3V3
- R81 pad 2: StackClear -> ~PortBReadHigh
- R91 pad 1: ~R1Out -> Net-(D42-Pad1)
- R91 pad 2: +3V3 -> GND
- R93 pad 1: ~R3Out -> Net-(D44-Pad1)
- R93 pad 2: +3V3 -> GND
- R94 pad 1: ~R4Out -> Net-(D45-Pad1)
- R94 pad 2: +3V3 -> GND
- R95 pad 1: Net-(R95-Pad1) -> Net-(D46-Pad1)
- R99 pad 1: ~R1Out -> Net-(D50-Pad1)
- R99 pad 2: +3V3 -> GND
- U11 pad 1: Net-(R47-Pad2) -> Net-(R61-Pad2)
- U11 pad 12: Net-(D40-Pad2) -> RAM_PAGE
- U11 pad 13: Net-(D39-Pad2) -> FLASHPAGE0
- U11 pad 14: Net-(D38-Pad2) -> FLASHPAGE1
- U11 pad 15: Net-(D37-Pad2) -> FLASHPAGE2
- U12 pad 1: ~GeneralRegisterLatch -> /ALU/Ins1
- U12 pad 10: GND -> Net-(U12-Pad10)
- U12 pad 11: Net-(U12-Pad11) -> Net-(R64-Pad2)
- U12 pad 12: RMAControl -> Net-(U12-Pad12)
- U12 pad 13: RJBControl -> Net-(U12-Pad13)
- U12 pad 14: R4Control -> Net-(U12-Pad14)
- U12 pad 15: R3Control -> Net-(U12-Pad15)
- U12 pad 16: R2Control -> /ALU/Ins9
- U12 pad 17: R1Control -> /ALU/Ins10
- U12 pad 18: DDR_Load -> /ALU/Ins11
- U12 pad 19: ~GeneralRegisterLatch -> /ALU/Ins12
- U12 pad 2: /ALU/Ins0 -> /ALU/Ins2
- U12 pad 20: +3V3 -> /ALU/Ins13
- U12 pad 3: /ALU/Ins1 -> /ALU/Ins3
- U12 pad 4: /ALU/Ins2 -> /ALU/Ins4
- U12 pad 5: /ALU/Ins3 -> /ALU/Ins5
- U12 pad 6: /ALU/Ins4 -> /ALU/Ins6
- U12 pad 7: /ALU/Ins5 -> /ALU/Ins7
- U12 pad 8: /ALU/Ins6 -> /ALU/Ins8
- U15 pad 1: ~StackOut -> ~PortEnable
- U15 pad 10: RegLatch -> GND
- U15 pad 11: ~I-O_RegisterLatch -> Net-(U15-Pad11)
- U15 pad 12: RegLatch -> Net-(U15-Pad12)
- U15 pad 13: /ALU/Ins7 -> Net-(U15-Pad13)
- U15 pad 14: +3V3 -> Net-(U15-Pad14)
- U15 pad 2: ~RamAddrEnable -> /ALU/Ins0
- U15 pad 3: ~CounterOutEnable -> /ALU/Ins1
- U15 pad 4: /ALU/Ins7 -> /ALU/Ins2
- U15 pad 5: /ALU/Ins7 -> /ALU/Ins3
- U15 pad 7: GND -> Net-(U15-Pad7)
- U15 pad 8: ~GeneralRegisterLatch -> Net-(U15-Pad8)
- U15 pad 9: Net-(U15-Pad6) -> Net-(U15-Pad9)
- U17 pad 1: /ProgramCounter/JB5 -> Net-(U17-Pad1)
- U17 pad 10: /ProgramCounter/JB6 -> RegLatch
- U17 pad 11: ~CounterLoad -> ~I-O_RegisterLatch
- U17 pad 12: Net-(U17-Pad12) -> RegLatch
- U17 pad 13: Net-(U17-Pad13) -> /ALU/Ins7
- U17 pad 14: CounterClear -> +3V3
- U17 pad 2: /ProgramCounter/PC5 -> Net-(U17-Pad2)
- U17 pad 3: /ProgramCounter/PC4 -> Net-(U17-Pad3)
- U17 pad 4: Net-(U16-Pad13) -> /ALU/Ins7
- U17 pad 5: Net-(U16-Pad12) -> /ALU/Ins7
- U17 pad 6: /ProgramCounter/PC6 -> Net-(U17-Pad6)
- U17 pad 7: /ProgramCounter/PC7 -> GND
- U17 pad 8: GND -> ~GeneralRegisterLatch
- U17 pad 9: /ProgramCounter/JB7 -> Net-(U17-Pad6)
- U18 pad 1: /ProgramCounter/JB9 -> /ProgramCounter/JB1
- U18 pad 10: /ProgramCounter/JB10 -> /ProgramCounter/JB2
- U18 pad 15: /ProgramCounter/JB8 -> /ProgramCounter/JB0
- U18 pad 2: /ProgramCounter/PC9 -> /ProgramCounter/PC1
- U18 pad 3: /ProgramCounter/PC8 -> /ProgramCounter/PC0
- U18 pad 4: Net-(U17-Pad13) -> Net-(R102-Pad2)
- U18 pad 5: Net-(U17-Pad12) -> CounterUp
- U18 pad 6: /ProgramCounter/PC10 -> /ProgramCounter/PC2
- U18 pad 7: /ProgramCounter/PC11 -> /ProgramCounter/PC3
- U18 pad 9: /ProgramCounter/JB11 -> /ProgramCounter/JB3
- U19 pad 1: /ProgramCounter/JB13 -> /ProgramCounter/JB5
- U19 pad 10: /ProgramCounter/JB14 -> /ProgramCounter/JB6
- U19 pad 15: /ProgramCounter/JB12 -> /ProgramCounter/JB4
- U19 pad 2: /ProgramCounter/PC13 -> /ProgramCounter/PC5
- U19 pad 3: /ProgramCounter/PC12 -> /ProgramCounter/PC4
- U19 pad 6: /ProgramCounter/PC14 -> /ProgramCounter/PC6
- U19 pad 7: /ProgramCounter/PC15 -> /ProgramCounter/PC7
- U19 pad 9: /ProgramCounter/JB15 -> /ProgramCounter/JB7
- U20 pad 1: ~CounterOutEnable -> /ProgramCounter/JB9
- U20 pad 10: GND -> /ProgramCounter/JB10
- U20 pad 11: /Memory/MA7 -> ~CounterLoad
- U20 pad 12: /Memory/MA6 -> Net-(U20-Pad12)
- U20 pad 13: /Memory/MA5 -> Net-(U20-Pad13)
- U20 pad 14: /Memory/MA4 -> CounterClear
- U20 pad 15: /Memory/MA3 -> /ProgramCounter/JB8
- U20 pad 16: /Memory/MA2 -> +3V3
- U20 pad 2: /ProgramCounter/PC0 -> /ProgramCounter/PC9
- U20 pad 3: /ProgramCounter/PC1 -> /ProgramCounter/PC8
- U20 pad 4: /ProgramCounter/PC2 -> Net-(U19-Pad13)
- U20 pad 5: /ProgramCounter/PC3 -> Net-(U19-Pad12)
- U20 pad 6: /ProgramCounter/PC4 -> /ProgramCounter/PC10
- U20 pad 7: /ProgramCounter/PC5 -> /ProgramCounter/PC11
- U20 pad 8: /ProgramCounter/PC6 -> GND
- U20 pad 9: /ProgramCounter/PC7 -> /ProgramCounter/JB11
- U21 pad 1: ~CounterOutEnable -> /ProgramCounter/JB13
- U21 pad 10: GND -> /ProgramCounter/JB14
- U21 pad 11: /Memory/MA15 -> ~CounterLoad
- U21 pad 12: /Memory/MA14 -> Net-(U21-Pad12)
- U21 pad 13: /Memory/MA13 -> Net-(U21-Pad13)
- U21 pad 14: /Memory/MA12 -> CounterClear
- U21 pad 15: /Memory/MA11 -> /ProgramCounter/JB12
- U21 pad 16: /Memory/MA10 -> +3V3
- U21 pad 2: /ProgramCounter/PC8 -> /ProgramCounter/PC13
- U21 pad 3: /ProgramCounter/PC9 -> /ProgramCounter/PC12
- U21 pad 4: /ProgramCounter/PC10 -> Net-(U20-Pad13)
- U21 pad 5: /ProgramCounter/PC11 -> Net-(U20-Pad12)
- U21 pad 6: /ProgramCounter/PC12 -> /ProgramCounter/PC14
- U21 pad 7: /ProgramCounter/PC13 -> /ProgramCounter/PC15
- U21 pad 8: /ProgramCounter/PC14 -> GND
- U21 pad 9: /ProgramCounter/PC15 -> /ProgramCounter/JB15
- U22 pad 1: /ALU/B1 -> ~CounterOutEnable
- U22 pad 10: /ALU/B2 -> GND
- U22 pad 11: ~StackLoad -> /Boot Flash/MA7
- U22 pad 12: Net-(U22-Pad12) -> /Boot Flash/MA6
- U22 pad 13: Net-(U22-Pad13) -> /Boot Flash/MA5
- U22 pad 14: StackClear -> /Boot Flash/MA4
- U22 pad 15: /ALU/B0 -> /Boot Flash/MA3
- U22 pad 16: +3V3 -> /Boot Flash/MA2
- U22 pad 2: /StackPointer/SP1 -> /ProgramCounter/PC0
- U22 pad 3: /StackPointer/SP0 -> /ProgramCounter/PC1
- U22 pad 4: StackDown -> /ProgramCounter/PC2
- U22 pad 5: StackUp -> /ProgramCounter/PC3
- U22 pad 6: /StackPointer/SP2 -> /ProgramCounter/PC4
- U22 pad 7: /StackPointer/SP3 -> /ProgramCounter/PC5
- U22 pad 8: GND -> /ProgramCounter/PC6
- U22 pad 9: /ALU/B3 -> /ProgramCounter/PC7
- U23 pad 1: /ALU/B5 -> ~CounterOutEnable
- U23 pad 10: /ALU/B6 -> GND
- U23 pad 11: ~StackLoad -> /Boot Flash/MA15
- U23 pad 12: Net-(U23-Pad12) -> /Boot Flash/MA14
- U23 pad 13: Net-(U23-Pad13) -> /Boot Flash/MA13
- U23 pad 14: StackClear -> /Boot Flash/MA12
- U23 pad 15: /ALU/B4 -> /Boot Flash/MA11
- U23 pad 16: +3V3 -> /Boot Flash/MA10
- U23 pad 2: /StackPointer/SP5 -> /ProgramCounter/PC8
- U23 pad 3: /StackPointer/SP4 -> /ProgramCounter/PC9
- U23 pad 4: Net-(U22-Pad13) -> /ProgramCounter/PC10
- U23 pad 5: Net-(U22-Pad12) -> /ProgramCounter/PC11
- U23 pad 6: /StackPointer/SP6 -> /ProgramCounter/PC12
- U23 pad 7: /StackPointer/SP7 -> /ProgramCounter/PC13
- U23 pad 8: GND -> /ProgramCounter/PC14
- U23 pad 9: /ALU/B7 -> /ProgramCounter/PC15
- U24 pad 1: /ALU/B9 -> /ALU/B1
- U24 pad 10: /ALU/B10 -> /ALU/B2
- U24 pad 15: /ALU/B8 -> /ALU/B0
- U24 pad 2: /StackPointer/SP9 -> /StackPointer/SP1
- U24 pad 3: /StackPointer/SP8 -> /StackPointer/SP0
- U24 pad 4: Net-(U23-Pad13) -> StackDown
- U24 pad 5: Net-(U23-Pad12) -> StackUp
- U24 pad 6: /StackPointer/SP10 -> /StackPointer/SP2
- U24 pad 7: /StackPointer/SP11 -> /StackPointer/SP3
- U24 pad 9: /ALU/B11 -> /ALU/B3
- U25 pad 1: /ALU/B13 -> /ALU/B5
- U25 pad 10: /ALU/B14 -> /ALU/B6
- U25 pad 15: /ALU/B12 -> /ALU/B4
- U25 pad 2: /StackPointer/SP13 -> /StackPointer/SP5
- U25 pad 3: /StackPointer/SP12 -> /StackPointer/SP4
- U25 pad 6: /StackPointer/SP14 -> /StackPointer/SP6
- U25 pad 7: /StackPointer/SP15 -> /StackPointer/SP7
- U25 pad 9: /ALU/B15 -> /ALU/B7
- U26 pad 1: ~StackOut -> /ALU/B9
- U26 pad 10: GND -> /ALU/B10
- U26 pad 11: /Memory/MA7 -> ~StackLoad
- U26 pad 12: /Memory/MA6 -> Net-(U26-Pad12)
- U26 pad 13: /Memory/MA5 -> Net-(U26-Pad13)
- U26 pad 14: /Memory/MA4 -> StackClear
- U26 pad 15: /Memory/MA3 -> /ALU/B8
- U26 pad 16: /Memory/MA2 -> +3V3
- U26 pad 2: /StackPointer/SP0 -> /StackPointer/SP9
- U26 pad 3: /StackPointer/SP1 -> /StackPointer/SP8
- U26 pad 4: /StackPointer/SP2 -> Net-(U25-Pad13)
- U26 pad 5: /StackPointer/SP3 -> Net-(U25-Pad12)
- U26 pad 6: /StackPointer/SP4 -> /StackPointer/SP10
- U26 pad 7: /StackPointer/SP5 -> /StackPointer/SP11
- U26 pad 8: /StackPointer/SP6 -> GND
- U26 pad 9: /StackPointer/SP7 -> /ALU/B11
- U29 pad 11: /Memory/MA15 -> /Boot Flash/MA15
- U29 pad 12: /Memory/MA14 -> /Boot Flash/MA14
- U29 pad 13: /Memory/MA13 -> /Boot Flash/MA13
- U29 pad 14: /Memory/MA12 -> /Boot Flash/MA12
- U29 pad 15: /Memory/MA11 -> /Boot Flash/MA11
- U29 pad 16: /Memory/MA10 -> /Boot Flash/MA10
- U29 pad 17: /Memory/MA9 -> /Boot Flash/MA9
- U29 pad 18: /Memory/MA8 -> /Boot Flash/MA8
- U30 pad 1: /Memory/MA3 -> /Boot Flash/MA3
- U30 pad 18: /Memory/MA8 -> /Boot Flash/MA8
- U30 pad 19: /Memory/MA9 -> /Boot Flash/MA9
- U30 pad 2: /Memory/MA4 -> /Boot Flash/MA4
- U30 pad 20: /Memory/MA10 -> /Boot Flash/MA10
- U30 pad 21: /Memory/MA11 -> /Boot Flash/MA11
- U30 pad 22: /Memory/MA12 -> /Boot Flash/MA12
- U30 pad 24: Net-(R88-Pad1) -> RAM_PAGE
- U30 pad 25: /Memory/MA13 -> /Boot Flash/MA13
- U30 pad 26: /Memory/MA14 -> /Boot Flash/MA14
- U30 pad 27: /Memory/MA15 -> /Boot Flash/MA15
- U30 pad 3: /Memory/MA5 -> /Boot Flash/MA5
- U30 pad 4: /Memory/MA6 -> /Boot Flash/MA6
- U30 pad 42: /Memory/MA0 -> /Boot Flash/MA0
- U30 pad 43: /Memory/MA1 -> /Boot Flash/MA1
- U30 pad 44: /Memory/MA2 -> /Boot Flash/MA2
- U30 pad 5: /Memory/MA7 -> /Boot Flash/MA7
- U33 pad 1: ~R3Out -> ~R1Out
- U33 pad 11: R3Control -> R1Control
- U35 pad 1: Net-(R95-Pad1) -> ~R3Out
- U35 pad 11: RJBControl -> R3Control
- U35 pad 12: /ProgramCounter/JB7 -> /ALU/OddR7
- U35 pad 13: /ProgramCounter/JB6 -> /ALU/OddR6
- U35 pad 14: /ProgramCounter/JB5 -> /ALU/OddR5
- U35 pad 15: /ProgramCounter/JB4 -> /ALU/OddR4
- U35 pad 16: /ProgramCounter/JB3 -> /ALU/OddR3
- U35 pad 17: /ProgramCounter/JB2 -> /ALU/OddR2
- U35 pad 18: /ProgramCounter/JB1 -> /ALU/OddR1
- U35 pad 19: /ProgramCounter/JB0 -> /ALU/OddR0
- U41 pad 1: ~R3Out -> ~R1Out
- U41 pad 11: R3Control -> R1Control
- U45 pad 1: Net-(R103-Pad1) -> Net-(R132-Pad1)
- U49 pad 1: ~MainRegRightOutput -> ~MainRegLeftOutput
- U49 pad 11: /ALU/EvenR7 -> /ALU/OddR7
- U49 pad 12: /ALU/EvenR6 -> /ALU/OddR6
- U49 pad 13: /ALU/EvenR5 -> /ALU/OddR5
- U49 pad 14: /ALU/EvenR4 -> /ALU/OddR4
- U49 pad 15: /ALU/EvenR3 -> /ALU/OddR3
- U49 pad 16: /ALU/EvenR2 -> /ALU/OddR2
- U49 pad 17: /ALU/EvenR1 -> /ALU/OddR1
- U49 pad 18: /ALU/EvenR0 -> /ALU/OddR0
- U49 pad 19: ~MainRegRightOutput -> ~MainRegLeftOutput
- U50 pad 1: ~MainRegRightOutput -> ~MainRegLeftOutput
- U50 pad 11: /ALU/EvenR15 -> /ALU/OddR15
- U50 pad 12: /ALU/EvenR14 -> /ALU/OddR14
- U50 pad 13: /ALU/EvenR13 -> /ALU/OddR13
- U50 pad 14: /ALU/EvenR12 -> /ALU/OddR12
- U50 pad 15: /ALU/EvenR11 -> /ALU/OddR11
- U50 pad 16: /ALU/EvenR10 -> /ALU/OddR10
- U50 pad 17: /ALU/EvenR9 -> /ALU/OddR9
- U50 pad 18: /ALU/EvenR8 -> /ALU/OddR8
- U50 pad 19: ~MainRegRightOutput -> ~MainRegLeftOutput
- U53 pad 11: /Memory/MA7 -> /Boot Flash/MA7
- U53 pad 12: /Memory/MA6 -> /Boot Flash/MA6
- U53 pad 13: /Memory/MA5 -> /Boot Flash/MA5
- U53 pad 14: /Memory/MA4 -> /Boot Flash/MA4
- U53 pad 15: /Memory/MA3 -> /Boot Flash/MA3
- U53 pad 16: /Memory/MA2 -> /Boot Flash/MA2
- U53 pad 17: /Memory/MA1 -> /Boot Flash/MA1
- U53 pad 18: /Memory/MA0 -> /Boot Flash/MA0
- U54 pad 11: /Memory/MA15 -> /Boot Flash/MA15
- U54 pad 12: /Memory/MA14 -> /Boot Flash/MA14
- U54 pad 13: /Memory/MA13 -> /Boot Flash/MA13
- U54 pad 14: /Memory/MA12 -> /Boot Flash/MA12
- U54 pad 15: /Memory/MA11 -> /Boot Flash/MA11
- U54 pad 16: /Memory/MA10 -> /Boot Flash/MA10
- U54 pad 17: /Memory/MA9 -> /Boot Flash/MA9
- U54 pad 18: /Memory/MA8 -> /Boot Flash/MA8
- U55 pad 1: ~RMALeftOutput -> ~RMARightOutput
- U55 pad 11: /ALU/OddR7 -> /ALU/EvenR7
- U55 pad 12: /ALU/OddR6 -> /ALU/EvenR6
- U55 pad 13: /ALU/OddR5 -> /ALU/EvenR5
- U55 pad 14: /ALU/OddR4 -> /ALU/EvenR4
- U55 pad 15: /ALU/OddR3 -> /ALU/EvenR3
- U55 pad 16: /ALU/OddR2 -> /ALU/EvenR2
- U55 pad 17: /ALU/OddR1 -> /ALU/EvenR1
- U55 pad 18: /ALU/OddR0 -> /ALU/EvenR0
- U55 pad 19: ~RMALeftOutput -> ~RMARightOutput
- U56 pad 1: ~RMALeftOutput -> ~RMARightOutput
- U56 pad 11: /ALU/OddR15 -> /ALU/EvenR15
- U56 pad 12: /ALU/OddR14 -> /ALU/EvenR14
- U56 pad 13: /ALU/OddR13 -> /ALU/EvenR13
- U56 pad 14: /ALU/OddR12 -> /ALU/EvenR12
- U56 pad 15: /ALU/OddR11 -> /ALU/EvenR11
- U56 pad 16: /ALU/OddR10 -> /ALU/EvenR10
- U56 pad 17: /ALU/OddR9 -> /ALU/EvenR9
- U56 pad 18: /ALU/OddR8 -> /ALU/EvenR8
- U56 pad 19: ~RMALeftOutput -> ~RMARightOutput
- U57 pad 1: ~RJBRightOutput -> ~RMALeftOutput
- U57 pad 11: /ALU/EvenR7 -> /ALU/OddR7
- U57 pad 12: /ALU/EvenR6 -> /ALU/OddR6
- U57 pad 13: /ALU/EvenR5 -> /ALU/OddR5
- U57 pad 14: /ALU/EvenR4 -> /ALU/OddR4
- U57 pad 15: /ALU/EvenR3 -> /ALU/OddR3
- U57 pad 16: /ALU/EvenR2 -> /ALU/OddR2
- U57 pad 17: /ALU/EvenR1 -> /ALU/OddR1
- U57 pad 18: /ALU/EvenR0 -> /ALU/OddR0
- U57 pad 19: ~RJBRightOutput -> ~RMALeftOutput
- U57 pad 2: /ProgramCounter/JB0 -> /Registers/RA0
- U57 pad 3: /ProgramCounter/JB1 -> /Registers/RA1
- U57 pad 4: /ProgramCounter/JB2 -> /Registers/RA2
- U57 pad 5: /ProgramCounter/JB3 -> /Registers/RA3
- U57 pad 6: /ProgramCounter/JB4 -> /Registers/RA4
- U57 pad 7: /ProgramCounter/JB5 -> /Registers/RA5
- U57 pad 8: /ProgramCounter/JB6 -> /Registers/RA6
- U57 pad 9: /ProgramCounter/JB7 -> /Registers/RA7
- U58 pad 1: ~RJBRightOutput -> ~RMALeftOutput
- U58 pad 11: /ALU/EvenR15 -> /ALU/OddR15
- U58 pad 12: /ALU/EvenR14 -> /ALU/OddR14
- U58 pad 13: /ALU/EvenR13 -> /ALU/OddR13
- U58 pad 14: /ALU/EvenR12 -> /ALU/OddR12
- U58 pad 15: /ALU/EvenR11 -> /ALU/OddR11
- U58 pad 16: /ALU/EvenR10 -> /ALU/OddR10
- U58 pad 17: /ALU/EvenR9 -> /ALU/OddR9
- U58 pad 18: /ALU/EvenR8 -> /ALU/OddR8
- U58 pad 19: ~RJBRightOutput -> ~RMALeftOutput
- U58 pad 2: /ProgramCounter/JB8 -> /Registers/RA8
- U58 pad 3: /ProgramCounter/JB9 -> /Registers/RA9
- U58 pad 4: /ProgramCounter/JB10 -> /Registers/RA10
- U58 pad 5: /ProgramCounter/JB11 -> /Registers/RA11
- U58 pad 6: /ProgramCounter/JB12 -> /Registers/RA12
- U58 pad 7: /ProgramCounter/JB13 -> /Registers/RA13
- U58 pad 8: /ProgramCounter/JB14 -> /Registers/RA14
- U58 pad 9: /ProgramCounter/JB15 -> /Registers/RA15
- U59 pad 1: ~RJBLeftOutput -> ~RJBRightOutput
- U59 pad 11: /ALU/OddR7 -> /ALU/EvenR7
- U59 pad 12: /ALU/OddR6 -> /ALU/EvenR6
- U59 pad 13: /ALU/OddR5 -> /ALU/EvenR5
- U59 pad 14: /ALU/OddR4 -> /ALU/EvenR4
- U59 pad 15: /ALU/OddR3 -> /ALU/EvenR3
- U59 pad 16: /ALU/OddR2 -> /ALU/EvenR2
- U59 pad 17: /ALU/OddR1 -> /ALU/EvenR1
- U59 pad 18: /ALU/OddR0 -> /ALU/EvenR0
- U59 pad 19: ~RJBLeftOutput -> ~RJBRightOutput
- U60 pad 1: ~RJBLeftOutput -> ~RJBRightOutput
- U60 pad 11: /ALU/OddR15 -> /ALU/EvenR15
- U60 pad 12: /ALU/OddR14 -> /ALU/EvenR14
- U60 pad 13: /ALU/OddR13 -> /ALU/EvenR13
- U60 pad 14: /ALU/OddR12 -> /ALU/EvenR12
- U60 pad 15: /ALU/OddR11 -> /ALU/EvenR11
- U60 pad 16: /ALU/OddR10 -> /ALU/EvenR10
- U60 pad 17: /ALU/OddR9 -> /ALU/EvenR9
- U60 pad 18: /ALU/OddR8 -> /ALU/EvenR8
- U60 pad 19: ~RJBLeftOutput -> ~RJBRightOutput
- U61 pad 1: /ALU/OddR15 -> ~RJBLeftOutput
- U61 pad 10: /ALU/OddR8 -> GND
- U61 pad 19: Net-(U61-Pad19) -> ~RJBLeftOutput
- U61 pad 2: Net-(U61-Pad2) -> /ProgramCounter/JB0
- U61 pad 20: ~ALU_Enable -> +3V3
- U61 pad 3: /ALU/OddR14 -> /ProgramCounter/JB1
- U61 pad 4: /ALU/OddR13 -> /ProgramCounter/JB2
- U61 pad 5: /ALU/OddR12 -> /ProgramCounter/JB3
- U61 pad 6: /ALU/OddR11 -> /ProgramCounter/JB4
- U61 pad 7: Net-(U61-Pad7) -> /ProgramCounter/JB5
- U61 pad 8: /ALU/OddR10 -> /ProgramCounter/JB6
- U61 pad 9: /ALU/OddR9 -> /ProgramCounter/JB7
Routing:
- net GND: track 0.00 -> 1996.6 mm, vias 0 -> 50
- net +3V3: track 0.00 -> 1823.4 mm, vias 0 -> 43
- net /ALU/B15: track 0.00 -> 681.9 mm, vias 0 -> 27
- net /ALU/B12: track 0.00 -> 676.6 mm, vias 0 -> 30
- net /ALU/B8: track 0.00 -> 636.9 mm, vias 0 -> 37
- net /ALU/B9: track 0.00 -> 631.1 mm, vias 0 -> 32
- net /ALU/B14: track 0.00 -> 631.1 mm, vias 0 -> 27
- net /ALU/B3: track 0.00 -> 622.9 mm, vias 0 -> 24
- net /ALU/B2: track 0.00 -> 613.0 mm, vias 0 -> 25
- net /ALU/B11: track 0.00 -> 612.5 mm, vias 0 -> 28
- net /ALU/B5: track 0.00 -> 607.2 mm, vias 0 -> 24
- net /ALU/B13: track 0.00 -> 605.3 mm, vias 0 -> 27
- net /ALU/B4: track 0.00 -> 603.7 mm, vias 0 -> 23
- net /ALU/B7: track 0.00 -> 603.5 mm, vias 0 -> 28
- net /ALU/B0: track 0.00 -> 591.0 mm, vias 0 -> 27
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- added copper zone on F.Cu, net +3V3
- added copper zone on B.Cu, net GND
Other:
- board size 160 x 100 mm -> 192 x 120 mm
- net class Default: clearance 0.2 -> 0.127; trace_width 0.25 -> 0.127; via_dia 0.8 -> 0.4; via_drill 0.4 -> 0.2
- net class Power added: clearance 0.2, trace_width 0.5, via_dia 0.8, via_drill 0.4
- rule trace_clearance: 0.2 -> 0.127
- rule trace_min: 0.2 -> 0.127
- rule via_min_drill: 0.3 -> 0.2
- board text added: "3.3V"
- board text added: "3.3V Interface Enable"
- board text added: "CLK"
- board text added: "Designed By John Wallis 2021"
- board text added: "Disable"
- board text added: "GND"
- board text added: "I2C CLK"
- board text added: "I2C CLK (3.3V)"
- board text added: "I2C Data"
- board text added: "I2C Data (3.3V)"
- board text added: "Instruction"
- board text added: "JLCJLCJLCJLC"
- board text added: "Little Endian"
- board text added: "Main Bus"
- board text added: "Parallel Port"
- board text added: "Port AH"
- board text added: "Port AL"
- board text added: "Port BH"
- board text added: "Port BL"
- board text added: "Program Counter"
- board text added: "Serpent Intercepter X16"
- board text added: "TCK"
- board text added: "TDI"
- board text added: "TDO"
- board text added: "TMS"
