File: S3-Kicad/S3_Schematic.sch (KiCad schematic (older format))
At the start: 109 parts, among them J4 Conn_02x05_Odd_Even, SW1 SW_Push, SW2 SW_Push, U1 NE555P, U10 74LS241, U11 74LS241, U12 AS6C1008-55PCN, U13 74LS574, U14 74LS574, U15 CD4029BEE4, U16 CD4029BEE4, U17 CD4029BEE4, U18 CD4029BEE4, U19 74LS241, U2 NE555P, U20 74LS241, U21 74LS574, U22 74LS574, U23 74LS574, U24 74HC574, U28 EPM7128slc84-15n, U3 NE555P, U4 74LS574, U5 74LS574, U6 CD4029BEE4, U7 CD4029BEE4, U8 CD4029BEE4, U9 CD4029BEE4

Commit message: registers bank
Parts:
- removed R10, R11, R12, R13, R19, R20, R21, R8, R9: 50K, Resistor_THT:R_Axial_DIN0207_L6.3mm_D2.5mm_P7.62mm_Horizontal, symbol S3_Schematic-rescue:R-Device-MAX7000CPU-Gen2-rescue
- removed U10, U11, U19, U20: 74LS241, Package_DIP:DIP-20_W7.62mm, symbol S3_Schematic-rescue:74LS241-74xx-MAX7000CPU-Gen2-rescue
- removed U13, U14, U22, U23, U4, U5, U? (x11): 74LS574, Package_DIP:DIP-20_W7.62mm, symbol S3_Schematic-rescue:74LS573-74xx-MAX7000CPU-Gen2-rescue
- removed U15, U16, U17, U18, U6, U7, U8, U9: CD4029BEE4, Package_DIP:DIP-16_W7.62mm, symbol S3_Schematic-rescue:CD4029BEE4-CPU_ics
- added R? (x8): 50K, symbol Device:R
- added R? (x3): 50k, symbol Device:R
- added U? (x16): 74HC541, symbol 74xx:74LS541
- added U? (x13): 74HC574, symbol S3_Schematic-rescue:74LS573-74xx-MAX7000CPU-Gen2-rescue
- added U? (x4): 74hc193, symbol 74xx:74LS193
- added U? (x2): 74LS541, symbol 74xx:74LS541
- U21: value 74LS574 -> 74HC574; footprint Package_DIP:DIP-20_W7.62mm -> (none)
Connections:
- net labels added: Acc0, Acc1, Acc10, Acc11, Acc12, Acc13, Acc14, Acc15, Acc2, Acc3, Acc4, Acc5, Acc6, Acc7, Acc8, Acc9, EvenR10, EvenR11, EvenR12, EvenR13, EvenR14, EvenR15, EvenR8, EvenR9, MA0, MA1, MA10, MA11, MA12, MA13, MA14, MA15, MA2, MA3, MA4, MA5, MA6, MA7, MA8, MA9, OddR10, OddR11, OddR12, OddR13, OddR14, OddR15, OddR8, OddR9, SP0, SP1, SP10, SP11, SP12, SP13, SP14, SP15, SP2, SP3, SP4, SP5, SP6, SP7, SP8, SP9, StackClear, StackDown, StackUp, ~CounterOutEnable, ~MainRegLeftOutput, ~MainRegOutputControl, ~MainRegRightOutput, ~RJBLeftOutput, ~RJBRightOutput, ~RMALeftOutput, ~RMARightOutput, ~RamAddrEnable, ~StackLoad, ~StackOut
- net labels removed: Count, CounterOutControl, CounterOutEnable, HIGHJumpRegLoad, HighStackJump, JumpEnable, LOWJumpRegLoad, LowStackJump, MainRegOutputControl, RAM_Addr_Enable, RAM_HighControl, RAM_LowControl, StackCount, StackCountDirection, StackOutControl
- wire segments 448 -> 285
- no-connect marks 10 -> 8
Other:
- note added: "Clock Module/Debounce\n"
- note added: "Configurable ALU"
- note added: "General Purpose Registers/Control"
- note added: "MicroCode Memory\nSRAM\nState Machine\nFlags/ClkSelector\nLEDS\nGPIO\nSERIAL INTERFACE/ISP"
- note added: "StackPointer\n"
- note removed: "Clock Module\n"
- note removed: "Counter Module"
- note removed: "General Purpose Registers"
- note removed: "LEDs/drivers"
- note removed: "RAM/Instructions"
- note removed: "Stack \nCounter"
- moved on the sheet: R1, R2, R28, R29, R3, R30, R31, R33, R34, R35, R36, R37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

Commit message: Most of CPU planned out
Parts:
- removed C1, C2, C4, C6: 10n, Capacitor_THT:C_Disc_D5.0mm_W2.5mm_P2.50mm, symbol S3_Schematic-rescue:C-Device-MAX7000CPU-Gen2-rescue
- removed C3, C5: 100n, Capacitor_THT:C_Disc_D5.0mm_W2.5mm_P2.50mm, symbol S3_Schematic-rescue:C-Device-MAX7000CPU-Gen2-rescue
- removed J4: Conn_02x05_Odd_Even, Connector_PinHeader_2.54mm:PinHeader_2x05_P2.54mm_Vertical, symbol S3_Schematic-rescue:Conn_02x05_Odd_Even-Connector_Generic-MAX7000CPU-Gen2-rescue
- removed R1, R2, R3, R5: 1K, Resistor_THT:R_Axial_DIN0207_L6.3mm_D2.5mm_P7.62mm_Horizontal, symbol S3_Schematic-rescue:R-Device-MAX7000CPU-Gen2-rescue
- removed R14, R15, R16, R17, R18: 50K, Resistor_THT:R_Axial_DIN0207_L6.3mm_D2.5mm_P7.62mm_Horizontal, symbol S3_Schematic-rescue:R-Device-MAX7000CPU-Gen2-rescue
- removed R4, R6: 1M, Resistor_THT:R_Axial_DIN0207_L6.3mm_D2.5mm_P7.62mm_Horizontal, symbol S3_Schematic-rescue:R-Device-MAX7000CPU-Gen2-rescue
- removed RV1: 1M, MAX7000CPU:SIP460W50P254L970H980Q3P, symbol S3_Schematic-rescue:R_POT-Device-MAX7000CPU-Gen2-rescue
- removed SW1, SW2: SW_Push, Button_Switch_THT:SW_PUSH_6mm, symbol S3_Schematic-rescue:SW_Push-Switch-MAX7000CPU-Gen2-rescue
- removed U1, U2, U3: NE555P, Package_DIP:DIP-8_W7.62mm, symbol S3_Schematic-rescue:NE555P-Timer-MAX7000CPU-Gen2-rescue
- removed U12: AS6C1008-55PCN, Package_DIP:DIP-32_W15.24mm, symbol S3_Schematic-rescue:AS6C1008-55PCN-CPU_ics
- removed U28: EPM7128slc84-15n, Package_LCC:PLCC-84_THT-Socket, symbol S3_Schematic-rescue:EPM7128slc84-15n-CPU_ics
- added C1, C2: 32p, symbol Device:C
- added J1: Conn_02x16_Counter_Clockwise, symbol Connector_Generic:Conn_02x16_Counter_Clockwise
- added J2: Conn_01x02_Male, symbol Connector:Conn_01x02_Male
- added R10: 1k, symbol Device:R
- added R100, R101, R102, R11, R12, R22, R23, R24, R25, R42, R43, R44, R46, R47, R48, R53, R54, R63, R72, R73, R74, R75, R76, R77, R78, R79, R80, R81, R82, R83, R84, R85, R86, R87, R88, R89, R90, R91, R92, R93, R94, R95, R96, R97, R98, R99: 50K, symbol Device:R
- added R13, R16, R20, R21, R26, R41, R45: 50k, symbol Device:R
- added R9: 2.2M, symbol Device:R
- added U1: SN74LVC1GX04DCKR, SOT65P210X110-6N, symbol Gen3Parts:SN74LVC1GX04DCKR
- added U12: CY62136EV30LL-45ZSXI, SOP80P1184X119-44N, symbol Gen3Parts:CY62136EV30LL-45ZSXI
- added U17, U19, U22, U3, U31, U33, U60, U62, U63: 74HC541, symbol 74xx:74LS541
- added U18, U20, U30, U32, U43: 74HC574, Package_DIP:DIP-20_W7.62mm, symbol S3_Schematic-rescue:74LS573-74xx-MAX7000CPU-Gen2-rescue
- added U2: SST39VF800A-70-4C-EKE, SOP50P2000X120-48N, symbol Gen3Parts:SST39VF800A-70-4C-EKE
- added U34: XC9572XL-10TQG100C, QFP50P1600X1600X160-100N, symbol Gen3Parts:XC9572XL-10TQG100C
- added U61, U64, U66, U67: 74HC595, symbol 74xx:74HC595
- added U65: 74HC00, symbol 74xx:74HC00
- added Y1: Crystal, symbol Device:Crystal
- U13, U14, U15, U16: renamed from U?; value 74LS541 -> 74HC541
- gave numbers to parts that had none: 73
Connections:
- net labels added: +3.3V, CB0, CB1, CB10, CB11, CB12, CB13, CB14, CB15, CB2, CB3, CB4, CB5, CB6, CB7, CB8, CB9, CLK, CMA0, CMA1, CMA10, CMA11, CMA12, CMA13, CMA14, CMA15, CMA2, CMA3, CMA4, CMA5, CMA6, CMA7, CMA8, CMA9, DDR_Load, JumpS1, JumpS2, P0, P1, P10, P11, P12, P13, P14, P15, P16, P17, P18, P19, P2, P20, P21, P22, P23, P24, P25, P26, P27, P28, P29, P3, P30, P31, P4, P5, P6, P7, P8, P9, PS\2_CLK_3.3V, PS\2_CLK_5V, PS\2_Data_3.3V, PS\2_Data_5V, PortAWriteHigh, PortAWriteLow, PortBWriteHigh, PortBWriteLow, ProgamDataLatch, ProgamSerialCLK, ProgamSerialData, RegLatch, State0, State1, State2, TCK_5V, TDI_5V, TDO_5V, TMS_5V, ~AHDD, ~ALDD, ~ALU_Enable, ~BHDD, ~BLDD, ~ChipMemWriteControl, ~GeneralRegisterLatch, ~I-O_RegisterLatch, ~MemOutEnable, ~MemWriteControl, ~PortAReadHigh, ~PortAReadLow, ~PortBReadHigh, ~PortBReadLow, ~PortEnable, ~ProgamEnable, ~ProgamSerialClear, ~ProgramWriteData, ~R1Out, ~R2Out, ~R3Out, ~R4Out
- net labels removed: +5V, CLK_Select, MemOutEnable, MemWriteControl, RA_H0, RA_H1, RA_H2, RA_H3, RA_H4, RA_H5, RA_H6, RA_H7, RA_L0, RA_L1, RA_L2, RA_L3, RA_L4, RA_L5, RA_L6, RA_L7, SlowCLK, UserCLK
- wire segments 285 -> 599
- no-connect marks 8 -> 10
Other:
- note added: "ALU"
- note added: "Clock"
- note added: "GPIO\n"
- note added: "LEDS/PULLS/Headers/Probepoints\nGPIO - DDR use other states\nBOOTLOADER?\nISP\nResistor buffers"
- note added: "Microcode Decoder"
- note added: "Programing Logic"
- note added: "RAM module"
- note removed: "Clock Module/Debounce\n"
- note removed: "Configurable ALU"
- note removed: "MicroCode Memory\nSRAM\nState Machine\nFlags/ClkSelector\nLEDS\nGPIO\nSERIAL INTERFACE/ISP"
- moved on the sheet: R1, R14, R15, R17, R18, R19, R2, R27, R28, R29, R3, R30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

Commit message: some weekend changes
Parts:
- removed R1, R2, R3, R33, R34, R35, R36, R37, R38, R39, R4, R40, R5, R6, R7, R8: 50K, Resistor_THT:R_Axial_DIN0207_L6.3mm_D2.5mm_P7.62mm_Horizontal, symbol S3_Schematic-rescue:R-Device-MAX7000CPU-Gen2-rescue
- removed R101, R102, R80: 50K, symbol Device:R
- removed U61, U64, U66, U67: 74HC595, symbol 74xx:74HC595
- added J?: Conn_02x04_Counter_Clockwise, symbol Connector_Generic:Conn_02x04_Counter_Clockwise
- added J?: Conn_01x04, symbol Connector_Generic:Conn_01x04
- added R? (x5): 50K, symbol Device:R
Connections:
- net ~ChipMemWriteControl is gone; now on net ProgramInsDisable: U3.12 (Y6)
- net +3V3: now also R?.1, R?.1, R?.1, R?.1
- net GND: now also J?.7 (Pin_7), R?.2
- net PS\2_CLK_3.3V: now also U3.13 (Y5); no longer U3.14 (Y4)
- net PS\2_CLK_5V: now also J?.6 (Pin_6)
- net PS\2_Data_3.3V: now also U3.14 (Y4); no longer U3.13 (Y5)
- net PS\2_Data_5V: now also J?.5 (Pin_5)
- net TCK: now also R?.2
- net TCK_5V: now also J?.4 (Pin_4)
- net TDI: now also R?.2
- net TDI_5V: now also J?.2 (Pin_2)
- net TDO: now also R?.2
- net TDO_5V: now also J?.3 (Pin_3)
- net TMS: now also R?.2
- net TMS_5V: now also J?.1 (Pin_1)
- net at U1.3 (X1): now also C1.1, R9.2, Y1.1
- net ProgramInsDisable: now reaches R31.1, U24.1 (OE)
- net at U43.12 (Q7): now also J?.4 (Pin_4)
- net at U43.13 (Q6): now also J?.3 (Pin_3)
- net at U43.14 (Q5): now also J?.2 (Pin_2)
- net at U43.15 (Q4): now also J?.1 (Pin_1)
- net ~ProgramWriteData renamed ProgramInstructDisable_5V
- net ProgramInstructDisable_5V: now also J?.8 (Pin_8), R?.1
Other:
- note added: "LEDS/PULLS/Headers/Probepoints"
- note removed: "LEDS/PULLS/Headers/Probepoints\nGPIO - DDR use other states\nBOOTLOADER?\nISP\nResistor buffers"
- moved on the sheet: J2, R100, R45, R95, R96, R97, R98, R99, U3

Commit message: Schematic Done
Parts:
- removed J1: Conn_02x16_Counter_Clockwise, symbol Connector_Generic:Conn_02x16_Counter_Clockwise
- removed J2: Conn_01x02_Male, symbol Connector:Conn_01x02_Male
- removed J?: Conn_02x04_Counter_Clockwise, symbol Connector_Generic:Conn_02x04_Counter_Clockwise
- removed J?: Conn_01x04, symbol Connector_Generic:Conn_01x04
- removed R100, R22, R23, R24, R25, R42, R43, R44, R46, R47, R48, R53, R54, R63, R64, R65, R66, R67, R68, R69, R70, R71, R72, R73, R74, R75, R76, R77, R78, R79, R81, R82, R83, R84, R85, R86, R87, R88, R89, R90, R91, R92, R93, R94, R95, R96, R97, R98, R99, R? (x5): 50K, symbol Device:R
- removed R15, R16, R17, R18, R19, R20, R21, R26, R27, R32, R41, R45: 50k, symbol Device:R
- removed R28, R29, R30, R31, R49, R50, R51, R52, R55, R56, R57, R58, R59, R60, R61, R62: 50K, Resistor_THT:R_Axial_DIN0207_L6.3mm_D2.5mm_P7.62mm_Horizontal, symbol S3_Schematic-rescue:R-Device-MAX7000CPU-Gen2-rescue
- removed U1: SN74LVC1GX04DCKR, SOT65P210X110-6N, symbol Gen3Parts:SN74LVC1GX04DCKR
- removed U10, U11, U4, U5, U6, U7, U8, U9: 74hc193, symbol 74xx:74LS193
- removed U12: CY62136EV30LL-45ZSXI, SOP80P1184X119-44N, symbol Gen3Parts:CY62136EV30LL-45ZSXI
- removed U13, U14, U15, U16, U17, U19, U22, U3, U31, U33, U44, U45, U46, U47, U48, U49, U50, U51, U52, U53, U54, U55, U56, U57, U58, U59, U60, U62: 74HC541, symbol 74xx:74LS541
- removed U18, U20, U24, U30, U32, U35, U43: 74HC574, Package_DIP:DIP-20_W7.62mm, symbol S3_Schematic-rescue:74LS573-74xx-MAX7000CPU-Gen2-rescue
- removed U2: SST39VF800A-70-4C-EKE, SOP50P2000X120-48N, symbol Gen3Parts:SST39VF800A-70-4C-EKE
- removed U21, U23, U25, U26, U27, U28, U29, U36, U37, U38, U39, U40, U41, U42: 74HC574, symbol S3_Schematic-rescue:74LS573-74xx-MAX7000CPU-Gen2-rescue
- removed U34: XC9572XL-10TQG100C, QFP50P1600X1600X160-100N, symbol Gen3Parts:XC9572XL-10TQG100C
- removed U65: 74HC00, symbol 74xx:74HC00
- added C10, C11, C12, C13, C14, C15, C16, C17, C18, C19, C20, C21, C22, C23, C24, C25, C26, C27, C28, C29, C3, C30, C31, C32, C33, C34, C35, C36, C37, C38, C39, C4, C40, C41, C42, C43, C44, C45, C46, C47, C48, C49, C5, C50, C51, C52, C53, C54, C55, C56, C57, C58, C59, C6, C60, C61, C62, C63, C64, C65, C66, C67, C68, C69, C7, C70, C8, C9: 100n, Capacitor_SMD:C_0805_2012Metric, symbol Device:C
- added J3: Conn_02x04_Counter_Clockwise, Connector_PinHeader_2.54mm:PinHeader_2x04_P2.54mm_Vertical, symbol Connector_Generic:Conn_02x04_Counter_Clockwise
- added J4, J5: Conn_01x02, Connector_PinHeader_2.54mm:PinHeader_1x02_P2.54mm_Vertical, symbol Connector_Generic:Conn_01x02
- added J6, J7: Conn_01x04, Connector_PinHeader_2.54mm:PinHeader_1x04_P2.54mm_Vertical, symbol Connector_Generic:Conn_01x04
- added J8: Conn_01x03, Connector_PinHeader_2.54mm:PinHeader_1x03_P2.54mm_Vertical, symbol Connector_Generic:Conn_01x03
- added R1, R2, R3, R4, R5, R6, R7, R8: 50K, Resistor_SMD:R_0805_2012Metric, symbol Device:R
- added U62: SN74LVC1GX04DCKR, Package_TO_SOT_SMD:SOT-363_SC-70-6_Handsoldering, symbol Gen3Parts:SN74LVC1GX04DCKR
- C1, C2: footprint (none) -> Capacitor_SMD:C_0805_2012Metric
- R10: value 1k -> 50K; footprint (none) -> Resistor_SMD:R_0805_2012Metric
- R11: value 50K -> 2.2M; footprint (none) -> Resistor_SMD:R_0805_2012Metric
- R12: value 50K -> 1k; footprint (none) -> Resistor_SMD:R_0805_2012Metric
- R13, R14: value 50k -> 50K; footprint (none) -> Resistor_SMD:R_0805_2012Metric
- R9: value 2.2M -> 50K; footprint (none) -> Resistor_SMD:R_0805_2012Metric
- U63: footprint (none) -> Package_SO:TSSOP-20_4.4x6.5mm_P0.65mm
- Y1: footprint (none) -> Crystal:Crystal_HC49-U_Vertical
Connections:
- net Ins0 is gone; now on net TMS_5V: U63.2 (A0)
- net Ins1 is gone; now on net TDI_5V: U63.3 (A1)
- net Ins2 is gone; now on net TDO_5V: U63.4 (A2)
- net Ins3 is gone; now on net TCK_5V: U63.5 (A3)
- net Ins4 is gone; now on net PS\2_Data_5V: U63.6 (A4)
- net Ins5 is gone; now on net PS\2_CLK_5V: U63.7 (A5)
- net Ins6 is gone; now on net ProgramInstructDisable_5V: U63.8 (A6)
- net ~CounterLoad is gone; now on net GND: R14.2
- net ~MemOutEnable is gone; now on net ProgramInstructDisable_5V: R13.1
- net ~PortAReadLow is gone; now on an unnamed net: R12.2
- net ~R1Out is gone; now on net TMS: U63.18 (Y0)
- net ~R2Out is gone; now on net PS\2_Data_3.3V: U63.14 (Y4)
- net ~R3Out is gone; now on net TDI: U63.17 (Y1)
- net ~R4Out is gone; now on net PS\2_CLK_3.3V: U63.13 (Y5)
- net ~RJBLeftOutput is gone; now on net TDO: U63.16 (Y2)
- net ~RJBRightOutput is gone; now on net ProgramInsDisable: U63.12 (Y6)
- net ~RMALeftOutput is gone; now on net TCK: U63.15 (Y3)
- net +3V3: now also R10.1, R9.1, C10.1, C11.1, C12.1, C13.1, C14.1, C15.1, C16.1, C17.1, C18.1, C19.1, C20.1, C21.1, C22.1, C23.1, C24.1, C25.1, C26.1, C27.1, C28.1, C29.1, C3.1, C30.1, C31.1, C32.1, C33.1, C34.1, C35.1, C36.1, C37.1, C38.1, C39.1, C4.1, C40.1, C41.1, C42.1, C43.1, C44.1, C45.1, C46.1, C47.1, C48.1, C49.1, C5.1, C50.1, C51.1, C52.1, C53.1, C54.1, C55.1, C56.1, C57.1, C58.1, C59.1, C6.1, C60.1, C61.1, C62.1, C63.1, C64.1, C65.1, C66.1, C67.1, C68.1, C69.1, C7.1, C70.1, C8.1, C9.1, J5.1 (Pin_1), J6.1 (Pin_1), J6.2 (Pin_2), J6.3 (Pin_3), J6.4 (Pin_4), J8.1 (Pin_1), R1.1, R2.1, R3.1, R4.1, R5.1, R6.1, R7.1, R8.1, U62.5 (VCC); no longer R11.1, R12.1, R13.2, R14.1
- net CLK: now also J8.3 (Pin_3), U62.6 (Y)
- net GND: now also R13.2, C10.2, C11.2, C12.2, C13.2, C14.2, C15.2, C16.2, C17.2, C18.2, C19.2, C20.2, C21.2, C22.2, C23.2, C24.2, C25.2, C26.2, C27.2, C28.2, C29.2, C3.2, C30.2, C31.2, C32.2, C33.2, C35.2, C36.2, C37.2, C38.2, C39.2, C4.2, C40.2, C41.2, C42.2, C43.2, C44.2, C45.2, C46.2, C47.2, C48.2, C49.2, C5.2, C50.2, C51.2, C52.2, C53.2, C54.2, C55.2, C56.2, C57.2, C58.2, C59.2, C6.2, C60.2, C61.2, C62.2, C63.2, C64.2, C65.2, C66.2, C67.2, C68.2, C69.2, C7.2, C70.2, C8.2, C9.2, J3.7 (Pin_7), J7.1 (Pin_1), J7.2 (Pin_2), J7.3 (Pin_3), J7.4 (Pin_4), J8.2 (Pin_2), U62.2 (GND)
- net PS\2_CLK_3.3V: now also J4.2 (Pin_2)
- net PS\2_CLK_5V: now also J3.6 (Pin_6), R6.2
- net PS\2_Data_3.3V: now also J4.1 (Pin_1)
- net PS\2_Data_5V: now also J3.5 (Pin_5), R5.2
- net ProgramInstructDisable_5V: now also J3.8 (Pin_8)
- net TCK: now also R10.2
- net TCK_5V: now also J3.4 (Pin_4), R4.2
- net TDI: now also R8.2
- net TDI_5V: now also J3.2 (Pin_2), R2.2
- net TDO: now also R9.2
- net TDO_5V: now also J3.3 (Pin_3), R3.2
- net TMS: now also R7.2
- net TMS_5V: now also J3.1 (Pin_1), R1.2
- net at C1.1, Y1.1: now also R11.2, U62.3 (X1); no longer R9.2
- net at C2.1, Y1.2: no longer R10.2
- net Ins7: no longer names the net of U63.9 (A7)
- net ~ALU_Enable: no longer names the net of U63.1 (G1), U63.19 (G2)
- net ~ALU_Enable: now also R14.1, J5.2 (Pin_2)
- net ~RMARightOutput: no longer names the net of U63.11 (Y7)
- new net: R11.1, R12.1, U62.4 (X2)
- no-connect marks 10 -> 2
Other:
- note added: "Headers/Probepoints\n"
- note removed: "ALU"
- note removed: "GPIO\n"
- note removed: "General Purpose Registers/Control"
- note removed: "LEDS/PULLS/Headers/Probepoints"
- note removed: "Microcode Decoder"
- note removed: "Program Counter\n"
- note removed: "RAM module"
- note removed: "StackPointer\n"

Commit message: Circuit Board Drafted (it could probably be improved)
Parts:
- added C71, C72, C73, C74, C75, C76, C77, C78: 100n, Capacitor_SMD:C_0805_2012Metric, symbol Device:C
- added J11: Conn_01x02, Connector_PinHeader_2.54mm:PinHeader_1x02_P2.54mm_Vertical, symbol Connector_Generic:Conn_01x02
- renumbered J3 to J1, J4 to J2, J5 to J3, J6 to J4, J7 to J5, J8 to J6, U62 to U1, U63 to U2
Connections:
- net +3V3: now also C71.1, C72.1, C73.1, C74.1, C75.1, C76.1, C77.1, C78.1
- net GND: now also C34.2, C71.2, C72.2, C73.2, C74.2, C75.2, C76.2, C77.2, C78.2
- net PS\2_CLK_5V: now also J11.2 (Pin_2)
- net PS\2_Data_5V: now also J11.1 (Pin_1)
