File: S3-Kicad/StackPointer.sch (KiCad schematic (older format))
At the start: 9 parts, among them U22 74hc193, U23 74hc193, U24 74hc193, U25 74hc193, U26 74HC541, U27 74HC541

Commit message: Circuit Board Drafted (it could probably be improved)
Parts:
- renumbered R80 to R110, R81 to R111, R82 to R112, U22 to U24, U23 to U25, U24 to U26, U25 to U27, U26 to U28, U27 to U29
Changed lines of the file:
@@
 $Descr A4 11693 8268
 encoding utf-8
-Sheet 5 8
+Sheet 5 9
 Title ""
 Date ""
@@
 P 5050 2600
 AR Path="/667BB40D" Ref="U?"  Part="1"
-AR Path="/636BC396/667BB40D" Ref="U23"  Part="1"
-F 0 "U23" H 4650 3250 50  0000 C CNN
+AR Path="/636BC396/667BB40D" Ref="U25"  Part="1"
+F 0 "U25" H 4650 3250 50  0000 C CNN
 F 1 "74hc193" H 4750 3150 50  0000 C CNN
 F 2 "Package_SO:TSSOP-16_4.4x5mm_P0.65mm" H 5050 2600 50  0001 C CNN
@@
 P 3600 3400
 AR Path="/667BB413" Ref="#PWR?"  Part="1"
-AR Path="/636BC396/667BB413" Ref="#PWR0151"  Part="1"
-F 0 "#PWR0151" H 3600 3150 50  0001 C CNN
+AR Path="/636BC396/667BB413" Ref="#PWR068"  Part="1"
+F 0 "#PWR068" H 3600 3150 50  0001 C CNN
 F 1 "GND" H 3600 3250 50  0000 C CNN
 F 2 "" H 3600 3400 50  0001 C CNN
@@
 P 5050 3400
 AR Path="/667BB419" Ref="#PWR?"  Part="1"
-AR Path="/636BC396/667BB419" Ref="#PWR0152"  Part="1"
-F 0 "#PWR0152" H 5050 3150 50  0001 C CNN
+AR Path="/636BC396/667BB419" Ref="#PWR069"  Part="1"
+F 0 "#PWR069" H 5050 3150 50  0001 C CNN
 F 1 "GND" H 5050 3250 50  0000 C CNN
 F 2 "" H 5050 3400 50  0001 C CNN
@@
 P 3600 2600
 AR Path="/667BB41F" Ref="U?"  Part="1"
-AR Path="/636BC396/667BB41F" Ref="U22"  Part="1"
-F 0 "U22" H 3200 3250 50  0000 C CNN
+AR Path="/636BC396/667BB41F" Ref="U24"  Part="1"
+F 0 "U24" H 3200 3250 50  0000 C CNN
 F 1 "74hc193" H 3300 3150 50  0000 C CNN
 F 2 "Package_SO:TSSOP-16_4.4x5mm_P0.65mm" H 3600 2600 50  0001 C CNN
@@
 P 7950 2600
 AR Path="/667BB42B" Ref="U?"  Part="1"
-AR Path="/636BC396/667BB42B" Ref="U25"  Part="1"
-F 0 "U25" H 7550 3250 50  0000 C CNN
+AR Path="/636BC396/667BB42B" Ref="U27"  Part="1"
+F 0 "U27" H 7550 3250 50  0000 C CNN
 F 1 "74hc193" H 7650 3150 50  0000 C CNN
 F 2 "Package_SO:TSSOP-16_4.4x5mm_P0.65mm" H 7950 2600 50  0001 C CNN
@@
 P 6500 3400
 AR Path="/667BB431" Ref="#PWR?"  Part="1"
-AR Path="/636BC396/667BB431" Ref="#PWR0153"  Part="1"
-F 0 "#PWR0153" H 6500 3150 50  0001 C CNN
+AR Path="/636BC396/667BB431" Ref="#PWR070"  Part="1"
+F 0 "#PWR070" H 6500 3150 50  0001 C CNN
 F 1 "GND" H 6500 3250 50  0000 C CNN
 F 2 "" H 6500 3400 50  0001 C CNN
@@
 P 7950 3400
 AR Path="/667BB437" Ref="#PWR?"  Part="1"
-AR Path="/636BC396/667BB437" Ref="#PWR0154"  Part="1"
-F 0 "#PWR0154" H 7950 3150 50  0001 C CNN
+AR Path="/636BC396/667BB437" Ref="#PWR071"  Part="1"
+F 0 "#PWR071" H 7950 3150 50  0001 C CNN
 F 1 "GND" H 7950 3250 50  0000 C CNN
 F 2 "" H 7950 3400 50  0001 C CNN
@@
 P 6500 2600
 AR Path="/667BB43D" Ref="U?"  Part="1"
-AR Path="/636BC396/667BB43D" Ref="U24"  Part="1"
-F 0 "U24" H 6100 3250 50  0000 C CNN
+AR Path="/636BC396/667BB43D" Ref="U26"  Part="1"
+F 0 "U26" H 6100 3250 50  0000 C CNN
 F 1 "74hc193" H 6200 3150 50  0000 C CNN
 F 2 "Package_SO:TSSOP-16_4.4x5mm_P0.65mm" H 6500 2600 50  0001 C CNN
@@
 P 4650 4700
 AR Path="/667BB465" Ref="U?"  Part="1"
-AR Path="/636BC396/667BB465" Ref="U26"  Part="1"
-F 0 "U26" H 4250 5450 50  0000 C CNN
+AR Path="/636BC396/667BB465" Ref="U28"  Part="1"
+F 0 "U28" H 4250 5450 50  0000 C CNN
 F 1 "74HC541" H 4350 5350 50  0000 C CNN
 F 2 "Package_SO:TSSOP-20_4.4x6.5mm_P0.65mm" H 4650 4700 50  0001 C CNN
@@
 P 7550 3850
 AR Path="/667BB46F" Ref="R?"  Part="1"
-AR Path="/636BC396/667BB46F" Ref="R80"  Part="1"
-F 0 "R80" V 7343 3850 50  0000 C CNN
+AR Path="/636BC396/667BB46F" Ref="R110"  Part="1"
+F 0 "R110" V 7343 3850 50  0000 C CNN
 F 1 "50K" V 7434 3850 50  0000 C CNN
 F 2 "Resistor_SMD:R_0805_2012Metric" V 7480 3850 50  0001 C CNN
@@
 P 7600 4000
 AR Path="/667BB47A" Ref="R?"  Part="1"
-AR Path="/636BC396/667BB47A" Ref="R81"  Part="1"
-F 0 "R81" V 7700 4000 50  0000 C CNN
+AR Path="/636BC396/667BB47A" Ref="R111"  Part="1"
+F 0 "R111" V 7700 4000 50  0000 C CNN
 F 1 "50K" V 7800 4000 50  0000 C CNN
 F 2 "Resistor_SMD:R_0805_2012Metric" V 7530 4000 50  0001 C CNN
@@
 P 7750 4000
 AR Path="/667BB481" Ref="#PWR?"  Part="1"
-AR Path="/636BC396/667BB481" Ref="#PWR0155"  Part="1"
-F 0 "#PWR0155" H 7750 3750 50  0001 C CNN
+AR Path="/636BC396/667BB481" Ref="#PWR075"  Part="1"
+F 0 "#PWR075" H 7750 3750 50  0001 C CNN
 F 1 "GND" H 7755 3827 50  0000 C CNN
 F 2 "" H 7750 4000 50  0001 C CNN
@@
 P 4650 5500
 AR Path="/667BB487" Ref="#PWR?"  Part="1"
-AR Path="/636BC396/667BB487" Ref="#PWR0156"  Part="1"
-F 0 "#PWR0156" H 4650 5250 50  0001 C CNN
+AR Path="/636BC396/667BB487" Ref="#PWR077"  Part="1"
+F 0 "#PWR077" H 4650 5250 50  0001 C CNN
 F 1 "GND" H 4655 5327 50  0000 C CNN
 F 2 "" H 4650 5500 50  0001 C CNN
@@
 P 6050 4700
 AR Path="/667BB48D" Ref="U?"  Part="1"
-AR Path="/636BC396/667BB48D" Ref="U27"  Part="1"
-F 0 "U27" H 5650 5450 50  0000 C CNN
+AR Path="/636BC396/667BB48D" Ref="U29"  Part="1"
+F 0 "U29" H 5650 5450 50  0000 C CNN
 F 1 "74HC541" H 5750 5350 50  0000 C CNN
 F 2 "Package_SO:TSSOP-20_4.4x6.5mm_P0.65mm" H 6050 4700 50  0001 C CNN
@@
 P 5400 5450
 AR Path="/667BB49A" Ref="R?"  Part="1"
-AR Path="/636BC396/667BB49A" Ref="R82"  Part="1"
-F 0 "R82" V 5193 5450 50  0000 C CNN
+AR Path="/636BC396/667BB49A" Ref="R112"  Part="1"
+F 0 "R112" V 5193 5450 50  0000 C CNN
 F 1 "50K" V 5284 5450 50  0000 C CNN
 F 2 "Resistor_SMD:R_0805_2012Metric" V 5330 5450 50  0001 C CNN
@@
 P 3600 1900
 AR Path="/667BB4F0" Ref="#PWR?"  Part="1"
-AR Path="/636BC396/667BB4F0" Ref="#PWR0157"  Part="1"
-F 0 "#PWR0157" H 3600 1750 50  0001 C CNN
+AR Path="/636BC396/667BB4F0" Ref="#PWR064"  Part="1"
+F 0 "#PWR064" H 3600 1750 50  0001 C CNN
 F 1 "+3.3V" H 3615 2073 50  0000 C CNN
 F 2 "" H 3600 1900 50  0001 C CNN
@@
 P 5050 1900
 AR Path="/667BB4F6" Ref="#PWR?"  Part="1"
-AR Path="/636BC396/667BB4F6" Ref="#PWR0158"  Part="1"
-F 0 "#PWR0158" H 5050 1750 50  0001 C CNN
+AR Path="/636BC396/667BB4F6" Ref="#PWR065"  Part="1"
+F 0 "#PWR065" H 5050 1750 50  0001 C CNN
 F 1 "+3.3V" H 5065 2073 50  0000 C CNN
 F 2 "" H 5050 1900 50  0001 C CNN
@@
 P 6500 1900
 AR Path="/667BB4FC" Ref="#PWR?"  Part="1"
-AR Path="/636BC396/667BB4FC" Ref="#PWR0159"  Part="1"
-F 0 "#PWR0159" H 6500 1750 50  0001 C CNN
+AR Path="/636BC396/667BB4FC" Ref="#PWR066"  Part="1"
+F 0 "#PWR066" H 6500 1750 50  0001 C CNN
 F 1 "+3.3V" H 6515 2073 50  0000 C CNN
 F 2 "" H 6500 1900 50  0001 C CNN
@@
 P 7950 1900
 AR Path="/667BB502" Ref="#PWR?"  Part="1"
-AR Path="/636BC396/667BB502" Ref="#PWR0160"  Part="1"
-F 0 "#PWR0160" H 7950 1750 50  0001 C CNN
+AR Path="/636BC396/667BB502" Ref="#PWR067"  Part="1"
+F 0 "#PWR067" H 7950 1750 50  0001 C CNN
 F 1 "+3.3V" H 7965 2073 50  0000 C CNN
 F 2 "" H 7950 1900 50  0001 C CNN
@@
 P 7700 3850
 AR Path="/667BB508" Ref="#PWR?"  Part="1"
-AR Path="/636BC396/667BB508" Ref="#PWR0161"  Part="1"
-F 0 "#PWR0161" H 7700 3700 50  0001 C CNN
+AR Path="/636BC396/667BB508" Ref="#PWR072"  Part="1"
+F 0 "#PWR072" H 7700 3700 50  0001 C CNN
 F 1 "+3.3V" H 7715 4023 50  0000 C CNN
 F 2 "" H 7700 3850 50  0001 C CNN
@@
 P 5250 5450
 AR Path="/667BB50E" Ref="#PWR?"  Part="1"
-AR Path="/636BC396/667BB50E" Ref="#PWR0162"  Part="1"
-F 0 "#PWR0162" H 5250 5300 50  0001 C CNN
+AR Path="/636BC396/667BB50E" Ref="#PWR076"  Part="1"
+F 0 "#PWR076" H 5250 5300 50  0001 C CNN
 F 1 "+3.3V" H 5200 5600 50  0000 C CNN
 F 2 "" H 5250 5450 50  0001 C CNN
@@
 P 4650 3900
 AR Path="/667BB514" Ref="#PWR?"  Part="1"
-AR Path="/636BC396/667BB514" Ref="#PWR0163"  Part="1"
-F 0 "#PWR0163" H 4650 3750 50  0001 C CNN
+AR Path="/636BC396/667BB514" Ref="#PWR073"  Part="1"
+F 0 "#PWR073" H 4650 3750 50  0001 C CNN
 F 1 "+3.3V" H 4665 4073 50  0000 C CNN
 F 2 "" H 4650 3900 50  0001 C CNN
@@
 P 6050 3900
 AR Path="/667BB51A" Ref="#PWR?"  Part="1"
-AR Path="/636BC396/667BB51A" Ref="#PWR0164"  Part="1"
-F 0 "#PWR0164" H 6050 3750 50  0001 C CNN
+AR Path="/636BC396/667BB51A" Ref="#PWR074"  Part="1"
+F 0 "#PWR074" H 6050 3750 50  0001 C CNN
 F 1 "+3.3V" H 6065 4073 50  0000 C CNN
 F 2 "" H 6050 3900 50  0001 C CNN
@@
 P 6050 5500
 AR Path="/667BB522" Ref="#PWR?"  Part="1"
-AR Path="/636BC396/667BB522" Ref="#PWR0165"  Part="1"
-F 0 "#PWR0165" H 6050 5250 50  0001 C CNN
+AR Path="/636BC396/667BB522" Ref="#PWR078"  Part="1"
+F 0 "#PWR078" H 6050 5250 50  0001 C CNN
 F 1 "GND" H 6055 5327 50  0000 C CNN
 F 2 "" H 6050 5500 50  0001 C CNN
